File: QualificationTestingAutomation/SchematicAutomation/MUXingsch.sch (KiCad schematic (older format))
At the start: 14 parts, among them U1 MC14067BDWG, U10 MC14051BDTR2G, U11 MC14051BDTR2G, U12 MC14051BDTR2G, U15 DS18B20_, U2 MC14051BDTR2G, U23 CD74HC4051E, U3 MC14051BDTR2G, U4 MC14051BDTR2G, U5 MC14051BDTR2G, U6 MC14051BDTR2G, U7 MC14051BDTR2G, U8 MC14051BDTR2G, U9 MC14051BDTR2G

Commit message: modified:   NMEAGUI/.classpath 	modified:   NMEAGUI/.settings/org.eclipse.jdt.core.prefs 	new file:   NMEAGUI/src/.classpath 	new file:   NMEAGUI/src/.project 	new file:   NMEAGUI/src/application/.gitignore 	modified:   QualificationTestingAutomation/SchematicAutomation/IO.bak 	modified:   QualificationTestingAutomation/SchematicAutomation/IO.sch 	modified:   QualificationTestingAutomation/SchematicAutomation/MUXingsch.bak 	new file:   QualificationTestingAutomation/SchematicAutomation/MUXingsch.pro 	modified:   QualificationTestingAutomation/SchematicAutomation/MUXingsch.sch 	modified:   QualificationTestingAutomation/SchematicAutomation/PWR.bak 	modified:   QualificationTestingAutomation/SchematicAutomation/PWR.sch 	modified:   QualificationTestingAutomation/SchematicAutomation/SchematicAutomation-cache.lib 	new file:   QualificationTestingAutomation/SchematicAutomation/_saved_MUXingsch.sch 	deleted:    QualificationTestingAutomation/SchematicAutomation/_saved_PWR.sch
Parts:
- removed U1: MC14067BDWG, MC14067BDWG:SOIC127P1030X265-24N, symbol MC14067BDWG:MC14067BDWG
- removed U10, U11, U12, U2, U3, U4, U5, U6, U7, U8, U9: MC14051BDTR2G, MC14051BDTR2G:SOP65P640X120-16N, symbol MC14051BDTR2G:MC14051BDTR2G
- removed U23: CD74HC4051E, digikey-footprints:DIP-16_W7.62mm, symbol dk_Interface-Analog-Switches-Multiplexers-Demultiplexers:CD74HC4051E
- added U?: CD74HC4067SM96, digikey-footprints:SSOP-24_W5.30mm, symbol dk_Interface-Analog-Switches-Multiplexers-Demultiplexers:CD74HC4067SM96
- added U?: LM339ADR, digikey-footprints:SOIC-14_W3.9mm, symbol dk_Linear-Comparators:LM339ADR
Connections:
- net labels added: +5V
- net labels removed: +12V
- wire segments 129 -> 130

Commit message: schematic is finished a few symbols were added, footprints are almost done, some work needs to be done on the connectors#
Parts:
- removed U15: DS18B20_, digikey-footprints:TO-92-3, symbol dk_Temperature-Sensors-Analog-and-Digital-Output:DS18B20_
- removed U?: CD74HC4067SM96, digikey-footprints:SSOP-24_W5.30mm, symbol dk_Interface-Analog-Switches-Multiplexers-Demultiplexers:CD74HC4067SM96
- removed U?: LM339ADR, digikey-footprints:SOIC-14_W3.9mm, symbol dk_Linear-Comparators:LM339ADR
Connections:
- net labels added: 1_ISO-Low, 1_J1708-RXD, 1_J1708-TXD, 2_ISO-Low, 2_J1708-RXD, 2_J1708-TXD, 3_CAN_MS_H, 3_ISO-Low, 3_J1708-RXD, 3_J1708-TXD, 4_ISO-Low, 4_J1708-RXD, 4_J1708-TXD, 5_ISO-Low, 5_J1708-RXD, 5_J1708-TXD, ISO-Low, J1708-RXD, J1708-TXD
- net labels removed: +5V, 1_J1708-RX, 1_J1708-TX, 1_OWB_MAIN, 1_OWB_SEC, 2_J1708-RX, 2_J1708-TX, 2_OWB_MAIN, 2_OWB_SEC, 3_CAN_MS_S, 3_J1708-RX, 3_J1708-TX, 3_OWB_MAIN, 3_OWB_SEC, 4_J1708-RX, 4_J1708-TX, 4_OWB_MAIN, 4_OWB_SEC, 5_J1708-RX, 5_J1708-TX, 5_OWB_MAIN, 5_OWB_SEC, GND, J1708-RX, J1708-TX, MUXA, MUXA1, MUXB, MUXC
- wire segments 130 -> 110
Changed lines of the file:
@@
 $Descr B 17000 11000
 encoding utf-8
-Sheet 3 6
+Sheet 3 18
 Title ""
 Date ""
@@
 5_CANLow
 Text GLabel 8550 8950 2    50   Input ~ 0
-ISO-K
+ISO-Low
 Wire Wire Line
 	8350 8950 8550 8950
 Text GLabel 7150 8750 0    50   Input ~ 0
-1_ISO-K
+1_ISO-Low
 Text GLabel 7150 8850 0    50   Input ~ 0
-2_ISO-K
+2_ISO-Low
 Text GLabel 7150 8950 0    50   Input ~ 0
-3_ISO-K
+3_ISO-Low
 Text GLabel 7150 9050 0    50   Input ~ 0
-4_ISO-K
+4_ISO-Low
 Text GLabel 7150 9150 0    50   Input ~ 0
-5_ISO-K
+5_ISO-Low
 Text GLabel 5550 8950 2    50   Input ~ 0
 CAN_MS_H
@@
 2_CAN_MS_H
 Text GLabel 4200 8950 0    50   Input ~ 0
-3_CAN_MS_S
+3_CAN_MS_H
 Text GLabel 4200 9050 0    50   Input ~ 0
 4_CAN_MS_H
@@
 5_SWC_BUS
 Text GLabel 8350 7250 2    50   Input ~ 0
-J1708-TX
+J1708-TXD
 Wire Wire Line
 	8150 7250 8350 7250
 Text GLabel 7000 7050 0    50   Input ~ 0
-1_J1708-TX
+1_J1708-TXD
 Text GLabel 7000 7150 0    50   Input ~ 0
-2_J1708-TX
+2_J1708-TXD
 Text GLabel 7000 7250 0    50   Input ~ 0
-3_J1708-TX
+3_J1708-TXD
 Text GLabel 7000 7350 0    50   Input ~ 0
-4_J1708-TX
+4_J1708-TXD
 Text GLabel 7000 7450 0    50   Input ~ 0
-5_J1708-TX
+5_J1708-TXD
 Text GLabel 2400 7150 2    50   Input ~ 0
-J1708-RX
+J1708-RXD
 Wire Wire Line
 	2200 7150 2400 7150
 Text GLabel 1150 6950 0    50   Input ~ 0
-1_J1708-RX
+1_J1708-RXD
 Text GLabel 1150 7050 0    50   Input ~ 0
-2_J1708-RX
+2_J1708-RXD
 Text GLabel 1150 7150 0    50   Input ~ 0
-3_J1708-RX
+3_J1708-RXD
 Text GLabel 1150 7250 0    50   Input ~ 0
-4_J1708-RX
+4_J1708-RXD
 Text GLabel 1150 7350 0    50   Input ~ 0
-5_J1708-RX
-$Comp
-L dk_Temperature-Sensors-Analog-and-Digital-Output:DS18B20_ U15
-U 1 1 5BB2A982
-P 1450 3850
-F 0 "U15" H 1578 3903 60  0000 L CNN
-F 1 "DS18B20_" H 1578 3797 60  0000 L CNN
-F 2 "digikey-footprints:TO-92-3" H 1650 4050 60  0001 L CNN
-F 3 "https://datasheets.maximintegrated.com/en/ds/DS18B20.pdf" H 1650 4150 60  0001 L CNN
-F 4 "DS18B20+-ND" H 1650 4250 60  0001 L CNN "Digi-Key_PN"
-F 5 "DS18B20+" H 1650 4350 60  0001 L CNN "MPN"
-F 6 "Sensors, Transducers" H 1650 4450 60  0001 L CNN "Category"
-F 7 "Temperature Sensors - Analog and Digital Output" H 1650 4550 60  0001 L CNN "Family"
-F 8 "https://datasheets.maximintegrated.com/en/ds/DS18B20.pdf" H 1650 4650 60  0001 L CNN "DK_Datasheet_Link"
-F 9 "/product-detail/en/maxim-integrated/DS18B20-/DS18B20--ND/956983" H 1650 4750 60  0001 L CNN "DK_Detail_Page"
-F 10 "SENSOR TEMPERATURE 1-WIRE TO92-3" H 1650 4850 60  0001 L CNN "Description"
-F 11 "Maxim Integrated" H 1650 4950 60  0001 L CNN "Manufacturer"
-F 12 "Active" H 1650 5050 60  0001 L CNN "Status"
-	1    1450 3850
-	-1   0    0    1
-$EndComp
-Wire Wire Line
-	1750 3850 1950 3850
-Wire Wire Line
-	1450 4150 1950 4150
-Wire Wire Line
-	1950 4150 1950 3850
-Connection ~ 1950 3850
-$Comp
-L power:GND #PWR056
-U 1 1 5BB3A9B5
-P 1450 3550
-F 0 "#PWR056" H 1450 3300 50  0001 C CNN
-F 1 "GND" H 1455 3377 50  0000 C CNN
-F 2 "" H 1450 3550 50  0001 C CNN
-F 3 "" H 1450 3550 50  0001 C CNN
-	1    1450 3550
-	-1   0    0    1
-$EndComp
-Text GLabel 5200 4150 2    50   Input ~ 0
-MUXA
-Text GLabel 5200 4250 2    50   Input ~ 0
-MUXB
-Text GLabel 5200 4350 2    50   Input ~ 0
-MUXC
-Wire Wire Line
-	5200 4350 4750 4350
-Wire Wire Line
-	5200 4250 4750 4250
-Wire Wire Line
-	5200 4150 4750 4150
-Text GLabel 5200 4050 2    50   Input ~ 0
-MUXA1
-Wire Wire Line
-	5200 4050 4750 4050
-Text GLabel 3400 4750 0    50   BiDi ~ 0
-5_OWB_MAIN
-Text GLabel 3400 4850 0    50   BiDi ~ 0
-5_OWB_SEC
-Wire Wire Line
-	3850 4050 3400 4050
-Wire Wire Line
-	3850 3950 3400 3950
-Text GLabel 3400 4550 0    50   BiDi ~ 0
-4_OWB_MAIN
-Text GLabel 3400 4650 0    50   BiDi ~ 0
-4_OWB_SEC
-Text GLabel 3400 4350 0    50   BiDi ~ 0
-3_OWB_MAIN
-Text GLabel 3400 4450 0    50   BiDi ~ 0
-3_OWB_SEC
-Wire Wire Line
-	3400 4150 3850 4150
-Wire Wire Line
-	3850 4250 3400 4250
-Wire Wire Line
-	3850 4350 3400 4350
-Wire Wire Line
-	3850 4450 3400 4450
-Text GLabel 3400 4150 0    50   BiDi ~ 0
-2_OWB_MAIN
-Text GLabel 3400 4250 0    50   BiDi ~ 0
-2_OWB_SEC
-Text GLabel 3400 4050 0    50   BiDi ~ 0
-1_OWB_MAIN
-Text GLabel 3400 3950 0    50   BiDi ~ 0
-1_OWB_SEC
-Wire Wire Line
-	3850 4550 3400 4550
-Wire Wire Line
-	3850 4650 3400 4650
-Wire Wire Line
-	3850 4750 3400 4750
-Wire Wire Line
-	3850 4850 3400 4850
-Wire Wire Line
-	4350 6050 4350 5850
-$Comp
-L power:GND #PWR055
-U 1 1 5BC72C5D
-P 4350 6050
-F 0 "#PWR055" H 4350 5800 50  0001 C CNN
-F 1 "GND" H 4355 5877 50  0000 C CNN
-F 2 "" H 4350 6050 50  0001 C CNN
-F 3 "" H 4350 6050 50  0001 C CNN
-	1    4350 6050
-	1    0    0    -1
-$EndComp
+5_J1708-RXD
 Wire Wire Line
 	2000 8700 2000 8800
@@
 	2200 7050 2200 7150
 Wire Wire Line
-	1950 3850 3850 3850
-$Comp
-L dk_Interface-Analog-Switches-Multiplexers-Demultiplexers:CD74HC4067SM96 U?
-U 1 1 5BB59507
-P 4350 4650
-F 0 "U?" H 4300 5950 60  0000 C CNN
-F 1 "CD74HC4067SM96" H 4300 5844 60  0000 C CNN
-F 2 "digikey-footprints:SSOP-24_W5.30mm" H 4550 4850 60  0001 L CNN
-F 3 "http://www.ti.com/lit/ds/symlink/cd74hc4067.pdf" H 4550 4950 60  0001 L CNN
-F 4 "296-9226-1-ND" H 4550 5050 60  0001 L CNN "Digi-Key_PN"
-F 5 "CD74HC4067SM96" H 4550 5150 60  0001 L CNN "MPN"
-F 6 "Integrated Circuits (ICs)" H 4550 5250 60  0001 L CNN "Category"
-F 7 "Interface - Analog Switches, Multiplexers, Demultiplexers" H 4550 5350 60  0001 L CNN "Family"
-F 8 "http://www.ti.com/lit/ds/symlink/cd74hc4067.pdf" H 4550 5450 60  0001 L CNN "DK_Datasheet_Link"
-F 9 "/product-detail/en/texas-instruments/CD74HC4067SM96/296-9226-1-ND/376978" H 4550 5550 60  0001 L CNN "DK_Detail_Page"
-F 10 "IC MUX/DEMUX 1X16 24SSOP" H 4550 5650 60  0001 L CNN "Description"
-F 11 "Texas Instruments" H 4550 5750 60  0001 L CNN "Manufacturer"
-F 12 "Active" H 4550 5850 60  0001 L CNN "Status"
-	1    4350 4650
-	1    0    0    -1
-$EndComp
-Wire Wire Line
 	5450 7350 5450 7250
 Wire Wire Line
@@
 Wire Wire Line
 	5450 7250 5450 7150
-$Comp
-L power:+5V #PWR?
-U 1 1 5BC13826
-P 4850 3550
-F 0 "#PWR?" H 4850 3400 50  0001 C CNN
-F 1 "+5V" H 4865 3723 50  0000 C CNN
-F 2 "" H 4850 3550 50  0001 C CNN
-F 3 "" H 4850 3550 50  0001 C CNN
-	1    4850 3550
-	1    0    0    -1
-$EndComp
-Wire Wire Line
-	4350 3550 4850 3550
-$Comp
-L dk_Linear-Comparators:LM339ADR U?
-U 1 1 5BE9CB2D
-P 10000 3400
-F 0 "U?" H 10341 3453 60  0000 L CNN
-F 1 "LM339ADR" H 10341 3347 60  0000 L CNN
-F 2 "digikey-footprints:SOIC-14_W3.9mm" H 10200 3600 60  0001 L CNN
-F 3 "http://www.ti.com/lit/ds/symlink/lm139a.pdf" H 10200 3700 60  0001 L CNN
-F 4 "296-6604-1-ND" H 10200 3800 60  0001 L CNN "Digi-Key_PN"
-F 5 "LM339ADR" H 10200 3900 60  0001 L CNN "MPN"
-F 6 "Integrated Circuits (ICs)" H 10200 4000 60  0001 L CNN "Category"
-F 7 "Linear - Comparators" H 10200 4100 60  0001 L CNN "Family"
-F 8 "http://www.ti.com/lit/ds/symlink/lm139a.pdf" H 10200 4200 60  0001 L CNN "DK_Datasheet_Link"
-F 9 "/product-detail/en/texas-instruments/LM339ADR/296-6604-1-ND/404682" H 10200 4300 60  0001 L CNN "DK_Detail_Page"
-F 10 "IC QUAD DIFF COMPARATOR 14 -SOIC" H 10200 4400 60  0001 L CNN "Description"
-F 11 "Texas Instruments" H 10200 4500 60  0001 L CNN "Manufacturer"
-F 12 "Active" H 10200 4600 60  0001 L CNN "Status"
-	1    10000 3400
-	1    0    0    -1
-$EndComp
 $EndSCHEMATC
