File: QualificationTestingAutomation/SchematicAutomation/USB.sch (KiCad schematic (older format))
At the start: 5 parts, among them IC1 TUSB2046B, J16 12401610E4_2A, Y5 6MHz

Commit message: Added Schematic Libraries
Parts:
- added C54: 1uF, symbol passive:CAP
- added R73, R74, R76, R77, R78, R80, R81, R82, R84, R85: 22, symbol passive:RESISTOR
- added R83, R88, R89: RESISTOR, symbol passive:RESISTOR
- added R86: 1.5K, symbol passive:RESISTOR
- added R87: 15K, symbol passive:RESISTOR
Connections:
- wire segments 38 -> 86
- no-connect marks 23 -> 21
Other:
- note added: "Maybe add a ferite beed to VCC"
