File: QualificationTestingAutomation/SchematicAutomation/USB.sch (KiCad schematic (older format))
At the start: 5 parts, among them IC1 TUSB2046B, J16 12401610E4_2A, Y5 6MHz

Commit message: C WPCB was started and the schematic is full, I am thinking of implementing the UART test using analog muxes.
Parts:
- C48, C49: footprint digikey-footprints:0603 -> smt:C-0603
- Y5: Digi-Key_PN (none) -> 535-10208-1-ND
Connections:
- net labels added: D0+, D0-
- net labels removed: DM0, DP0
- wire segments 32 -> 38
Changed lines of the file:
@@
 $Descr A4 11693 8268
 encoding utf-8
-Sheet 18 18
+Sheet 16 16
 Title ""
 Date ""
@@
 F 1 "6MHz" H 6850 3827 50  0000 C CNN
 F 2 "crystals:HC49UP" H 6850 3650 50  0001 C CNN
-F 3 "~" H 6850 3650 50  0001 C CNN
+F 3 "https://abracon.com/Resonators/abls.pdf" H 6850 3650 50  0001 C CNN
+F 4 " 535-10208-1-ND " H 0   0   50  0001 C CNN "Digi-Key_PN"
 	1    6850 3650
 	1    0    0    -1
@@
 U 1 1 5BE6E91E
 P 6650 3750
-F 0 "C48" H 6542 3708 60  0000 R CNB
-F 1 "20pF" H 6542 3803 45  0000 R CNN
-F 2 "digikey-footprints:0603" H 6685 3595 40  0001 L CNN
+F 0 "C48" H 6950 3800 60  0000 R CNB
+F 1 "20pF" H 6600 3850 45  0000 R CNN
+F 2 "smt:C-0603" H 6685 3595 40  0001 L CNN
 F 3 "" H 6650 3850 60  0001 C CNN
 F 4 "-" H 6690 3915 45  0001 L CNN "Part"
@@
 F 0 "C49" H 7108 3892 60  0000 L CNB
 F 1 "20pF" H 7108 3797 45  0000 L CNN
-F 2 "digikey-footprints:0603" H 7035 3695 40  0001 L CNN
+F 2 "smt:C-0603" H 7035 3695 40  0001 L CNN
 F 3 "" H 7000 3950 60  0001 C CNN
 F 4 "-" H 7040 4015 45  0001 L CNN "Part"
@@
 Wire Wire Line
 	6800 3950 7000 3950
-Wire Wire Line
-	6350 3850 6650 3850
-Connection ~ 6650 3850
 Wire Wire Line
 	4350 3750 4250 3750
@@
 DM4
 Text Label 4350 3450 2    50   ~ 0
-DP0
+D0+
 Text Label 4350 3550 2    50   ~ 0
-DM0
+D0-
 Wire Wire Line
 	4350 4150 4300 4150
@@
 $EndComp
 Wire Wire Line
-	6350 3950 6650 3950
+	6350 3950 6400 3950
 Connection ~ 6650 3950
 $Comp
@@
 F 1 "12401610E4_2A" H 2450 5401 60  0000 C CNN
 F 2 "digikey-footprints:USB_Type_C_Female__12401610E4_2A" H 2650 4600 60  0001 L CNN
-F 3 "https://media.digikey.com/pdf/Data%20Sheets/Amphenol%20PDFs/12401610E4%232A_Dwg.pdf" H 2650 4700 60  0001 L CNN
+F 3 "" H 2650 4700 60  0001 L CNN
 F 4 "12401610E4#2ACT-ND" H 2650 4800 60  0001 L CNN "Digi-Key_PN"
 F 5 "12401610E4#2A" H 2650 4900 60  0001 L CNN "MPN"
@@
 $EndComp
 Text Label 2950 4400 0    50   ~ 0
-DM0
+D0-
 Text Label 2950 4300 0    50   ~ 0
-DP0
+D0+
 Text Label 1950 4400 2    50   ~ 0
-DP0
+D0+
 Text Label 1950 4300 2    50   ~ 0
-DM0
+D0-
 $Comp
 L power:GND #PWR0300
 U 1 1 5BE72082
-P 2950 4900
-F 0 "#PWR0300" H 2950 4650 50  0001 C CNN
-F 1 "GND" H 2955 4727 50  0000 C CNN
-F 2 "" H 2950 4900 50  0001 C CNN
-F 3 "" H 2950 4900 50  0001 C CNN
-	1    2950 4900
+P 3050 4900
+F 0 "#PWR0300" H 3050 4650 50  0001 C CNN
+F 1 "GND" H 3055 4727 50  0000 C CNN
+F 2 "" H 3050 4900 50  0001 C CNN
+F 3 "" H 3050 4900 50  0001 C CNN
+	1    3050 4900
 	1    0    0    -1
 $EndComp
@@
 L power:GND #PWR0301
 U 1 1 5BE720B3
-P 2950 3800
-F 0 "#PWR0301" H 2950 3550 50  0001 C CNN
-F 1 "GND" H 2955 3627 50  0000 C CNN
-F 2 "" H 2950 3800 50  0001 C CNN
-F 3 "" H 2950 3800 50  0001 C CNN
-	1    2950 3800
+P 3050 3800
+F 0 "#PWR0301" H 3050 3550 50  0001 C CNN
+F 1 "GND" H 3150 3800 50  0000 C CNN
+F 2 "" H 3050 3800 50  0001 C CNN
+F 3 "" H 3050 3800 50  0001 C CNN
+	1    3050 3800
 	1    0    0    -1
 $EndComp
@@
 L power:GND #PWR0302
 U 1 1 5BE720E4
-P 1950 3800
-F 0 "#PWR0302" H 1950 3550 50  0001 C CNN
-F 1 "GND" H 1955 3627 50  0000 C CNN
-F 2 "" H 1950 3800 50  0001 C CNN
-F 3 "" H 1950 3800 50  0001 C CNN
-	1    1950 3800
+P 1850 3800
+F 0 "#PWR0302" H 1850 3550 50  0001 C CNN
+F 1 "GND" H 1750 3800 50  0000 C CNN
+F 2 "" H 1850 3800 50  0001 C CNN
+F 3 "" H 1850 3800 50  0001 C CNN
+	1    1850 3800
 	1    0    0    -1
 $EndComp
@@
 L power:GND #PWR0303
 U 1 1 5BE72115
-P 1950 4900
-F 0 "#PWR0303" H 1950 4650 50  0001 C CNN
-F 1 "GND" H 1955 4727 50  0000 C CNN
-F 2 "" H 1950 4900 50  0001 C CNN
-F 3 "" H 1950 4900 50  0001 C CNN
-	1    1950 4900
+P 1850 4900
+F 0 "#PWR0303" H 1850 4650 50  0001 C CNN
+F 1 "GND" H 1855 4727 50  0000 C CNN
+F 2 "" H 1850 4900 50  0001 C CNN
+F 3 "" H 1850 4900 50  0001 C CNN
+	1    1850 4900
 	1    0    0    -1
 $EndComp
@@
 NoConn ~ 2950 4700
 NoConn ~ 2950 4800
+Wire Wire Line
+	3050 3800 2950 3800
+Wire Wire Line
+	1950 3800 1850 3800
+Wire Wire Line
+	2950 4900 3050 4900
+Wire Wire Line
+	1950 4900 1850 4900
+Wire Wire Line
+	6350 3850 6400 3850
+Wire Wire Line
+	6400 3850 6400 3950
+Connection ~ 6400 3950
+Wire Wire Line
+	6400 3950 6650 3950
 $EndSCHEMATC

Commit message: Basis for the software
Connections:
- wire segments 38 -> 35
Changed lines of the file:
@@
 	-1   0    0    1
 $EndComp
-Wire Wire Line
-	6350 3650 6650 3650
-Connection ~ 6650 3650
-Wire Wire Line
-	6650 3650 6700 3650
-Wire Wire Line
-	7000 3750 6350 3750
-Wire Wire Line
-	7100 3750 7000 3750
-Connection ~ 7000 3750
 $Comp
 L passive:CAP C49
@@
 Wire Wire Line
 	6650 3850 6650 3950
-Wire Wire Line
-	6650 3950 6800 3950
-Connection ~ 6800 3950
-Wire Wire Line
-	6800 3950 7000 3950
 Wire Wire Line
 	4350 3750 4250 3750
@@
 Wire Wire Line
 	3150 4600 2950 4600
-Connection ~ 3150 4100
 $Comp
 L power:+5V #PWR0305
@@
 Wire Wire Line
 	1750 4100 1750 4600
-Connection ~ 1750 4100
 Wire Wire Line
 	1950 4600 1750 4600
@@
 Wire Wire Line
 	6400 3950 6650 3950
+Wire Wire Line
+	6350 3650 6700 3650
+Wire Wire Line
+	6350 3750 7100 3750
+Wire Wire Line
+	6650 3950 7000 3950
 $EndSCHEMATC
