File: QualificationTestingAutomation/SchematicAutomation/USB.sch (KiCad schematic (older format))
At the start: 21 parts, among them IC1 TUSB2046B, J16 12401610E4_2A, Y5 6MHz

Commit message: CLEANED UP THE SCHEMATICS ADDED NEADED FIXES FOUND ON THE BOARD
Parts:
- removed R89: RESISTOR, symbol passive:RESISTOR
- added R? (x8): 15K, symbol passive:RESISTOR
- R73, R74, R76, R77, R78, R80, R81, R82, R84, R85: value 22 -> 22R
- R83: value RESISTOR -> 1.5K
- R88: value RESISTOR -> 15K
Connections:
- wire segments 86 -> 105
- no-connect marks 21 -> 17
Other:
- note added: "SHOULD WE STICK WITH USB C/ IF NOT CHANGE THE CONNECTOR TOO HARD TO SOLDER"

Commit message: USB test instrument support and SCPI support were added to the FW
Parts:
- gave numbers to parts that had none: 8
Changed lines of the file:
@@
 DP2
 $Comp
-L passive:RESISTOR R?
+L passive:RESISTOR R151
 U 1 1 5BC525CF
 P 8450 4500
-F 0 "R?" V 8412 4553 60  0000 L CNB
+F 0 "R151" V 8412 4553 60  0000 L CNB
 F 1 "15K" V 8503 4553 40  0000 L CNN
 F 2 "" H 8450 4360 40  0001 C CNN
@@
 $EndComp
 $Comp
-L passive:RESISTOR R?
+L passive:RESISTOR R155
 U 1 1 5BC52722
 P 8750 4600
-F 0 "R?" V 8712 4653 60  0000 L CNB
+F 0 "R155" V 8712 4653 60  0000 L CNB
 F 1 "15K" V 8803 4653 40  0000 L CNN
 F 2 "" H 8750 4460 40  0001 C CNN
@@
 $EndComp
 $Comp
-L passive:RESISTOR R?
+L passive:RESISTOR R152
 U 1 1 5BC549F1
 P 8450 4900
-F 0 "R?" V 8412 4953 60  0000 L CNB
+F 0 "R152" V 8412 4953 60  0000 L CNB
 F 1 "15K" V 8503 4953 40  0000 L CNN
 F 2 "" H 8450 4760 40  0001 C CNN
@@
 $EndComp
 $Comp
-L passive:RESISTOR R?
+L passive:RESISTOR R156
 U 1 1 5BC56CD8
 P 8750 5000
-F 0 "R?" V 8712 5053 60  0000 L CNB
+F 0 "R156" V 8712 5053 60  0000 L CNB
 F 1 "15K" V 8803 5053 40  0000 L CNN
 F 2 "" H 8750 4860 40  0001 C CNN
@@
 $EndComp
 $Comp
-L passive:RESISTOR R?
+L passive:RESISTOR R153
 U 1 1 5BC58FC5
 P 8450 5400
-F 0 "R?" V 8412 5453 60  0000 L CNB
+F 0 "R153" V 8412 5453 60  0000 L CNB
 F 1 "15K" V 8503 5453 40  0000 L CNN
 F 2 "" H 8450 5260 40  0001 C CNN
@@
 $EndComp
 $Comp
-L passive:RESISTOR R?
+L passive:RESISTOR R157
 U 1 1 5BC5B2AE
 P 8750 5500
-F 0 "R?" V 8712 5553 60  0000 L CNB
+F 0 "R157" V 8712 5553 60  0000 L CNB
 F 1 "15K" V 8803 5553 40  0000 L CNN
 F 2 "" H 8750 5360 40  0001 C CNN
@@
 $EndComp
 $Comp
-L passive:RESISTOR R?
+L passive:RESISTOR R154
 U 1 1 5BC5D5A9
 P 8450 5800
-F 0 "R?" V 8412 5853 60  0000 L CNB
+F 0 "R154" V 8412 5853 60  0000 L CNB
 F 1 "15K" V 8503 5853 40  0000 L CNN
 F 2 "" H 8450 5660 40  0001 C CNN
@@
 $EndComp
 $Comp
-L passive:RESISTOR R?
+L passive:RESISTOR R158
 U 1 1 5BC5F894
 P 8750 5900
-F 0 "R?" V 8712 5953 60  0000 L CNB
+F 0 "R158" V 8712 5953 60  0000 L CNB
 F 1 "15K" V 8803 5953 40  0000 L CNN
 F 2 "" H 8750 5760 40  0001 C CNN
@@
 	8650 6000 8450 6000
 $Comp
-L power:GND #PWR?
+L power:GND #PWR0284
 U 1 1 5BC82D67
 P 8650 6200
-F 0 "#PWR?" H 8650 5950 50  0001 C CNN
+F 0 "#PWR0284" H 8650 5950 50  0001 C CNN
 F 1 "GND" H 8655 6027 50  0000 C CNN
 F 2 "" H 8650 6200 50  0001 C CNN
@@
 $EndComp
 $Comp
-L power:GND #PWR?
+L power:GND #PWR0286
 U 1 1 5BC82DD2
 P 8250 5600
-F 0 "#PWR?" H 8250 5350 50  0001 C CNN
+F 0 "#PWR0286" H 8250 5350 50  0001 C CNN
 F 1 "GND" H 8255 5427 50  0000 C CNN
 F 2 "" H 8250 5600 50  0001 C CNN
@@
 $EndComp
 $Comp
-L power:GND #PWR?
+L power:GND #PWR0287
 U 1 1 5BC85D05
 P 8200 5100
-F 0 "#PWR?" H 8200 4850 50  0001 C CNN
+F 0 "#PWR0287" H 8200 4850 50  0001 C CNN
 F 1 "GND" H 8205 4927 50  0000 C CNN
 F 2 "" H 8200 5100 50  0001 C CNN
@@
 $EndComp
 $Comp
-L power:GND #PWR?
+L power:GND #PWR0288
 U 1 1 5BC88C38
 P 8200 4700
-F 0 "#PWR?" H 8200 4450 50  0001 C CNN
+F 0 "#PWR0288" H 8200 4450 50  0001 C CNN
 F 1 "GND" H 8205 4527 50  0000 C CNN
 F 2 "" H 8200 4700 50  0001 C CNN
