File: QualificationTestingAutomation/SchematicAutomation/PWR.sch (KiCad schematic (older format))
At the start: 69 parts, among them J13 Barrel_Jack_MountingPin, J14 Banana Jack, J15 Banana Jack, Q1 ULN2003ADR, Q2 ULN2003ADR, U4 TPS563210, U5 TPS563210, U6 LM2776

Commit message: Basis for the software
Connections:
- wire segments 279 -> 240
Changed lines of the file:
@@
 	1    0    0    -1
 $EndComp
-Wire Wire Line
-	1800 2950 2300 2950
-Connection ~ 2300 2950
-Wire Wire Line
-	2300 2950 2700 2950
-Connection ~ 2700 2950
-Wire Wire Line
-	2700 2950 3150 2950
-Connection ~ 3150 2950
-Wire Wire Line
-	3150 2950 3650 2950
-Connection ~ 3650 2950
-Wire Wire Line
-	3650 2950 4100 2950
-Connection ~ 4100 2950
-Wire Wire Line
-	4100 2950 4600 2950
-Connection ~ 4600 2950
-Wire Wire Line
-	4600 2950 5150 2950
-Wire Wire Line
-	5150 2950 5600 2950
-Connection ~ 5600 2950
-Wire Wire Line
-	5600 2950 6100 2950
-Connection ~ 6100 2950
-Wire Wire Line
-	6100 2950 6550 2950
-Connection ~ 6550 2950
-Wire Wire Line
-	6550 2950 7050 2950
-Wire Wire Line
-	1800 3250 2300 3250
-Connection ~ 2300 3250
-Wire Wire Line
-	2300 3250 2700 3250
-Connection ~ 2700 3250
-Wire Wire Line
-	2700 3250 3150 3250
-Connection ~ 3150 3250
-Wire Wire Line
-	3150 3250 3650 3250
-Connection ~ 3650 3250
-Wire Wire Line
-	3650 3250 4100 3250
-Connection ~ 4100 3250
-Wire Wire Line
-	4100 3250 4600 3250
-Connection ~ 4600 3250
-Wire Wire Line
-	4600 3250 5150 3250
-Wire Wire Line
-	5150 3250 5600 3250
-Connection ~ 5600 3250
-Wire Wire Line
-	5600 3250 6100 3250
-Connection ~ 6100 3250
-Wire Wire Line
-	6100 3250 6550 3250
-Connection ~ 6550 3250
-Wire Wire Line
-	6550 3250 7050 3250
 $Comp
 L Device:C C29
@@
 $EndComp
 Wire Wire Line
-	5700 2350 6200 2350
-Connection ~ 6200 2350
-Wire Wire Line
-	6200 2350 6750 2350
-Connection ~ 6750 2350
-Wire Wire Line
-	6750 2350 7200 2350
-Connection ~ 7200 2350
-Wire Wire Line
-	7200 2350 7700 2350
-Connection ~ 7700 2350
-Wire Wire Line
-	7700 2350 8150 2350
-Connection ~ 8150 2350
-Wire Wire Line
-	8150 2350 8650 2350
-Connection ~ 8650 2350
-Wire Wire Line
-	8650 2350 9000 2350
-Wire Wire Line
-	5700 2650 6200 2650
-Connection ~ 6200 2650
-Wire Wire Line
-	6200 2650 6750 2650
-Connection ~ 6750 2650
-Wire Wire Line
-	6750 2650 7200 2650
-Connection ~ 7200 2650
-Wire Wire Line
-	7200 2650 7700 2650
-Connection ~ 7700 2650
-Wire Wire Line
-	7700 2650 8150 2650
-Connection ~ 8150 2650
-Wire Wire Line
-	8150 2650 8650 2650
-Connection ~ 8650 2650
-Wire Wire Line
-	8650 2650 9000 2650
-Wire Wire Line
 	9000 2350 9000 2300
 Connection ~ 9000 2350
@@
 	9000 2650 9000 2700
 Connection ~ 9000 2650
-Connection ~ 1800 2950
-Wire Wire Line
-	1800 3250 1350 3250
-Connection ~ 1800 3250
-Connection ~ 5150 3250
-Connection ~ 5150 2950
 Text GLabel 2550 6050 3    50   Input ~ 0
 1_Vin
@@
 Connection ~ 3500 5350
 Wire Wire Line
-	3500 5350 4150 5350
-Wire Wire Line
 	2250 5450 2250 5350
 Wire Wire Line
@@
 Wire Wire Line
 	3250 6050 3500 6050
-Connection ~ 3500 6050
 $Comp
 L dk_Diodes-Zener-Single:1N5231BTR Z3
@@
 Wire Wire Line
 	5600 6050 5900 6050
-Connection ~ 5900 6050
 Wire Wire Line
 	5600 5500 5600 5350
@@
 Wire Wire Line
 	6850 6100 7100 6100
-Connection ~ 7100 6100
 $Comp
 L power:+5V #PWR033
@@
 	1    0    0    -1
 $EndComp
-Connection ~ 4150 5350
-Wire Wire Line
-	4150 5350 4400 5350
 Wire Wire Line
 	2450 5450 2450 5250
@@
 Connection ~ 11700 5150
 Wire Wire Line
-	11700 5150 12350 5150
-Wire Wire Line
 	10450 5250 10450 5150
 Wire Wire Line
@@
 Wire Wire Line
 	11450 5850 11700 5850
-Connection ~ 11700 5850
 $Comp
 L dk_Diodes-Zener-Single:1N5231BTR Z8
@@
 Wire Wire Line
 	13800 5850 14100 5850
-Connection ~ 14100 5850
 Wire Wire Line
 	13800 5300 13800 5150
@@
 Wire Wire Line
 	15050 5900 15300 5900
-Connection ~ 15300 5900
 $Comp
 L power:+5V #PWR054
@@
 	1    0    0    -1
 $EndComp
-Connection ~ 12350 5150
-Wire Wire Line
-	12350 5150 12600 5150
 Wire Wire Line
 	10650 5250 10650 5050
@@
 Text GLabel 15600 5900 3    50   Input ~ 0
 5_GarminPWR
-Wire Wire Line
-	7050 2950 7550 2950
-Connection ~ 7050 2950
 $Comp
 L passive:CAP C44
@@
 Wire Wire Line
 	7550 3150 7550 3250
-Wire Wire Line
-	7550 3250 7050 3250
-Connection ~ 7050 3250
 Wire Wire Line
 	16200 5200 16200 5250
@@
 $EndComp
 Wire Wire Line
-	4100 1950 4450 1950
-Wire Wire Line
 	4500 1950 4500 2050
 Connection ~ 4100 1950
@@
 $EndComp
 Wire Wire Line
-	1300 2950 1800 2950
-Wire Wire Line
 	1550 1950 850  1950
 $Comp
@@
 	1    0    0    -1
 $EndComp
-Connection ~ 4450 1950
-Wire Wire Line
-	4450 1950 4500 1950
+Wire Wire Line
+	3500 5350 4400 5350
+Wire Wire Line
+	11700 5150 12600 5150
+Wire Wire Line
+	4100 1950 4500 1950
+Wire Wire Line
+	5700 2350 9000 2350
+Wire Wire Line
+	5700 2650 9000 2650
+Wire Wire Line
+	1300 2950 7550 2950
+Wire Wire Line
+	1350 3250 7550 3250
 $EndSCHEMATC
