File: QualificationTestingAutomation/SchematicAutomation/PWR.sch (KiCad schematic (older format))
At the start: 28 parts, among them J14 Conn_01x02, J2 Barrel_Jack_MountingPin, J3 Conn_01x02, U13 LD1117S33TR_SOT223, U14 LD1117S50TR_SOT223

Commit message: modified:   NMEAGUI/.classpath 	modified:   NMEAGUI/.settings/org.eclipse.jdt.core.prefs 	new file:   NMEAGUI/src/.classpath 	new file:   NMEAGUI/src/.project 	new file:   NMEAGUI/src/application/.gitignore 	modified:   QualificationTestingAutomation/SchematicAutomation/IO.bak 	modified:   QualificationTestingAutomation/SchematicAutomation/IO.sch 	modified:   QualificationTestingAutomation/SchematicAutomation/MUXingsch.bak 	new file:   QualificationTestingAutomation/SchematicAutomation/MUXingsch.pro 	modified:   QualificationTestingAutomation/SchematicAutomation/MUXingsch.sch 	modified:   QualificationTestingAutomation/SchematicAutomation/PWR.bak 	modified:   QualificationTestingAutomation/SchematicAutomation/PWR.sch 	modified:   QualificationTestingAutomation/SchematicAutomation/SchematicAutomation-cache.lib 	new file:   QualificationTestingAutomation/SchematicAutomation/_saved_MUXingsch.sch 	deleted:    QualificationTestingAutomation/SchematicAutomation/_saved_PWR.sch
Parts:
- added Q?: ULN2003ADR, digikey-footprints:SOIC-16_W3.90mm, symbol dk_Transistors-Bipolar-BJT-Arrays:ULN2003ADR
- added RLY? (x5): G5LE-14_DC5, digikey-footprints:Relay_THT_G5LE-14, symbol dk_Power-Relays-Over-2-Amps:G5LE-14_DC5
- added S? (x2): ATE1D-2M3-10-Z, digikey-footprints:Switch_Toggle_ATE1D-2M3-10-Z, symbol dk_Toggle-Switches:ATE1D-2M3-10-Z
- added Z? (x5): 1N5231BTR, digikey-footprints:DO-35, symbol dk_Diodes-Zener-Single:1N5231BTR
Connections:
- net labels added: +VSW, 1_REL, 1_Vin, 2_REL, 2_Vin, 3_REL, 3_Vin, 4_REL, 4_Vin, 5_REL, 5_Vin
- wire segments 72 -> 145

Commit message: schematic is finished a few symbols were added, footprints are almost done, some work needs to be done on the connectors#
Parts:
- removed S?: ATE1D-2M3-10-Z, digikey-footprints:Switch_Toggle_ATE1D-2M3-10-Z, symbol dk_Toggle-Switches:ATE1D-2M3-10-Z
- added C28, C30: 2.2uF, digikey-footprints:0603, symbol passive:CAP
- added C31: 1uF, digikey-footprints:0603, symbol passive:CAP
- added C44: 4.7uF, digikey-footprints:0603, symbol passive:CAP
- added Q2: ULN2003ADR, digikey-footprints:SOIC-16_W3.90mm, symbol dk_Transistors-Bipolar-BJT-Arrays:ULN2003ADR
- added RLY10, RLY6, RLY7, RLY8, RLY9: G5LE-14_DC5, digikey-footprints:Relay_THT_G5LE-14, symbol dk_Power-Relays-Over-2-Amps:G5LE-14_DC5
- added S2: ATE1D-2M3-10-Z, digikey-footprints:Switch_Toggle_ATE1D-2M3-10-Z, symbol dk_Toggle-Switches:ATE1D-2M3-10-Z
- added U6: LM2776, digikey-footprints:SOT-23-6, symbol Power_Management:LM2776
- added Z10, Z6, Z7, Z8, Z9: 1N5231BTR, digikey-footprints:DO-35, symbol dk_Diodes-Zener-Single:1N5231BTR
- C10: renamed from C4; footprint digikey-footprints:0805 -> digikey-footprints:0603
- C11: renamed from C?; footprint digikey-footprints:1206 -> digikey-footprints:1210
- C12: renamed from C5; footprint digikey-footprints:0805 -> digikey-footprints:0603
- C13: renamed from C6; footprint digikey-footprints:0805 -> digikey-footprints:0603
- C14: renamed from C; footprint digikey-footprints:0805 -> digikey-footprints:0603
- C15: renamed from C8; footprint digikey-footprints:0805 -> digikey-footprints:0603
- C16: renamed from C10; footprint digikey-footprints:0805 -> digikey-footprints:0603
- C17: renamed from C; footprint digikey-footprints:1206 -> digikey-footprints:1210
- C18: renamed from C12; footprint digikey-footprints:0805 -> digikey-footprints:0603
- C19: renamed from C7; footprint digikey-footprints:0805 -> digikey-footprints:0603
- C20: renamed from C14; footprint digikey-footprints:0805 -> digikey-footprints:0603
- C21: renamed from C9; footprint digikey-footprints:0805 -> digikey-footprints:0603
- C22: renamed from C16; footprint digikey-footprints:0805 -> digikey-footprints:0603
- C23: renamed from C11; footprint digikey-footprints:0805 -> digikey-footprints:0603
- C24: renamed from C18; footprint digikey-footprints:0805 -> digikey-footprints:0603
- C25: renamed from C13; footprint digikey-footprints:0805 -> digikey-footprints:0603
- C26: renamed from C15; footprint digikey-footprints:0805 -> digikey-footprints:0603
- C27: renamed from C17; footprint digikey-footprints:0805 -> digikey-footprints:0603
- C29: renamed from C19; footprint digikey-footprints:0805 -> digikey-footprints:0603
- C6: renamed from C1; footprint digikey-footprints:0805 -> digikey-footprints:0603
- C7: renamed from C?; footprint digikey-footprints:0805 -> digikey-footprints:0603
- C8: renamed from C2; footprint digikey-footprints:0805 -> digikey-footprints:0603
- C9: renamed from C3; footprint digikey-footprints:0805 -> digikey-footprints:0603
- gave numbers to parts that had none: 12
- renumbered J2 to J13, J3 to J15, U13 to U4, U14 to U5
Connections:
- net labels added: -3V3, -VSW, 1_GarminPWR, 2_GarminPWR, 3_GarminPWR, 4_GarminPWR, 5_GarminPWR, VDC
- net labels removed: +VDC
- wire segments 145 -> 242
- no-connect marks 0 -> 8
Other:
- moved on the sheet: U4, U5

Commit message: C WPCB was started and the schematic is full, I am thinking of implementing the UART test using analog muxes.
Parts:
- C10, C12, C13, C14, C15, C16, C18, C19, C20, C21, C22, C23, C24, C25, C26, C27, C29, C6, C7, C8, C9: footprint digikey-footprints:0603 -> smt:C-0603
- C11: footprint digikey-footprints:1210 -> digikey-footprints:0805
- C17: footprint digikey-footprints:1210 -> digikey-footprints:1206
- C28, C30, C31, C44: footprint digikey-footprints:0603 -> smt:C-0805
- J13: footprint (none) -> Connectors:Barrel_Jack_CUI_PJ-102AH; DK_Datasheet_Link (none) -> https://www.cui.com/product/resource/digikeypdf/pj-037a.pdf; Digi-Key_PN (none) -> CP-037A-ND
- J14, J15: value Conn_01x02 -> Banana Jack; footprint (none) -> Connectors:Banana_Jack_2Pin; Description (none) -> The hole has a diameter of about 5.2mm (fits standard 4mm b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
- U4, U5: footprint Package_TO_SOT_SMD:SOT-223-3_TabPin2 -> TO_SOT_Packages_SMD:SOT-223-3_TabPin2
Connections:
- wire segments 242 -> 240
Changed lines of the file:
@@
 $Descr B 17000 11000
 encoding utf-8
-Sheet 5 18
+Sheet 5 16
 Title ""
 Date ""
@@
 F 0 "U4" H 2700 1142 50  0000 C CNN
 F 1 "LD1117S33TR_SOT223" H 2700 1051 50  0000 C CNN
-F 2 "Package_TO_SOT_SMD:SOT-223-3_TabPin2" H 2700 1100 50  0001 C CNN
+F 2 "TO_SOT_Packages_SMD:SOT-223-3_TabPin2" H 2700 1100 50  0001 C CNN
 F 3 "http://www.st.com/st-web-ui/static/active/en/resource/technical/document/datasheet/CD00000544.pdf" H 2800 650 50  0001 C CNN
 	1    2700 900
@@
 F 0 "C7" H 2215 1146 50  0000 L CNN
 F 1 "100nF" H 2215 1055 50  0000 L CNN
-F 2 "digikey-footprints:0603" H 2138 950 50  0001 C CNN
+F 2 "smt:C-0603" H 2138 950 50  0001 C CNN
 F 3 "~" H 2100 1100 50  0001 C CNN
 	1    2100 1100
@@
 F 0 "C11" H 3465 1146 50  0000 L CNN
 F 1 "100uF" H 3465 1055 50  0000 L CNN
-F 2 "digikey-footprints:1210" H 3388 950 50  0001 C CNN
+F 2 "digikey-footprints:0805" H 3388 950 50  0001 C CNN
 F 3 "~" H 3350 1100 50  0001 C CNN
 	1    3350 1100
@@
 F 0 "C14" H 4365 1196 50  0000 L CNN
 F 1 "100nF" H 4365 1105 50  0000 L CNN
-F 2 "digikey-footprints:0603" H 4288 1000 50  0001 C CNN
+F 2 "smt:C-0603" H 4288 1000 50  0001 C CNN
 F 3 "~" H 4250 1150 50  0001 C CNN
 	1    4250 1150
@@
 F 0 "C17" H 5615 1196 50  0000 L CNN
 F 1 "100uF" H 5615 1105 50  0000 L CNN
-F 2 "digikey-footprints:1210" H 5538 1000 50  0001 C CNN
+F 2 "digikey-footprints:1206" H 5538 1000 50  0001 C CNN
 F 3 "~" H 5500 1150 50  0001 C CNN
 	1    5500 1150
@@
 F 0 "U5" H 4850 1192 50  0000 C CNN
 F 1 "LD1117S50TR_SOT223" H 4850 1101 50  0000 C CNN
-F 2 "Package_TO_SOT_SMD:SOT-223-3_TabPin2" H 4850 1150 50  0001 C CNN
+F 2 "TO_SOT_Packages_SMD:SOT-223-3_TabPin2" H 4850 1150 50  0001 C CNN
 F 3 "http://www.st.com/st-web-ui/static/active/en/resource/technical/document/datasheet/CD00000544.pdf" H 4950 700 50  0001 C CNN
 	1    4850 950
@@
 AR Path="/5BA2CD36/5BE1D7EC" Ref="J15"  Part="1"
 F 0 "J15" H 10530 2292 50  0000 L CNN
-F 1 "Conn_01x02" H 10530 2201 50  0000 L CNN
-F 2 "" H 10450 2300 50  0001 C CNN
+F 1 "Banana Jack" H 10530 2201 50  0000 L CNN
+F 2 "Connectors:Banana_Jack_2Pin" H 10450 2300 50  0001 C CNN
 F 3 "~" H 10450 2300 50  0001 C CNN
+F 4 "The hole has a diameter of about 5.2mm (fits standard 4mm banana plugs), the cap on the front has an outside diameter of about 11.6mm and length of 15.2mm. Diameter of the screw is 3.8mm. The mounting key is about 4 x 5.4mm." H 0   0   50  0001 C CNN "Description"
 	1    10450 2300
 	1    0    0    -1
@@
 F 0 "J13" H 1005 1517 50  0000 C CNN
 F 1 "Barrel_Jack_MountingPin" H 1005 1426 50  0000 C CNN
-F 2 "" H 1000 1160 50  0001 C CNN
-F 3 "~" H 1000 1160 50  0001 C CNN
+F 2 "Connectors:Barrel_Jack_CUI_PJ-102AH" H 1000 1160 50  0001 C CNN
+F 3 "https://www.cui.com/product/resource/digikeypdf/pj-037a.pdf" H 1000 1160 50  0001 C CNN
+F 4 " CP-037A-ND " H 0   0   50  0001 C CNN "Digi-Key_PN"
+F 5 "https://www.cui.com/product/resource/digikeypdf/pj-037a.pdf" H 0   0   50  0001 C CNN "DK_Datasheet_Link"
 	1    950  1200
 	1    0    0    -1
@@
 AR Path="/5BA2CD36/5BE1D81B" Ref="J14"  Part="1"
 F 0 "J14" H 9530 2492 50  0000 L CNN
-F 1 "Conn_01x02" H 9530 2401 50  0000 L CNN
-F 2 "" H 9450 2500 50  0001 C CNN
+F 1 "Banana Jack" H 9530 2401 50  0000 L CNN
+F 2 "Connectors:Banana_Jack_2Pin" H 9450 2500 50  0001 C CNN
 F 3 "~" H 9450 2500 50  0001 C CNN
+F 4 "The hole has a diameter of about 5.2mm (fits standard 4mm banana plugs), the cap on the front has an outside diameter of about 11.6mm and length of 15.2mm. Diameter of the screw is 3.8mm. The mounting key is about 4 x 5.4mm." H 0   0   50  0001 C CNN "Description"
 	1    9450 2500
 	1    0    0    -1
@@
 F 0 "C24" H 7165 3146 50  0000 L CNN
 F 1 ".01uF" H 7165 3055 50  0000 L CNN
-F 2 "digikey-footprints:0603" H 7088 2950 50  0001 C CNN
+F 2 "smt:C-0603" H 7088 2950 50  0001 C CNN
 F 3 "~" H 7050 3100 50  0001 C CNN
 	1    7050 3100
@@
 F 0 "C22" H 6665 3146 50  0000 L CNN
 F 1 ".01uF" H 6665 3055 50  0000 L CNN
-F 2 "digikey-footprints:0603" H 6588 2950 50  0001 C CNN
+F 2 "smt:C-0603" H 6588 2950 50  0001 C CNN
 F 3 "~" H 6550 3100 50  0001 C CNN
 	1    6550 3100
@@
 F 0 "C20" H 6215 3146 50  0000 L CNN
 F 1 ".01uF" H 6215 3055 50  0000 L CNN
-F 2 "digikey-footprints:0603" H 6138 2950 50  0001 C CNN
+F 2 "smt:C-0603" H 6138 2950 50  0001 C CNN
 F 3 "~" H 6100 3100 50  0001 C CNN
 	1    6100 3100
@@
 F 0 "C18" H 5715 3146 50  0000 L CNN
 F 1 ".01uF" H 5715 3055 50  0000 L CNN
-F 2 "digikey-footprints:0603" H 5638 2950 50  0001 C CNN
+F 2 "smt:C-0603" H 5638 2950 50  0001 C CNN
 F 3 "~" H 5600 3100 50  0001 C CNN
 	1    5600 3100
@@
 F 0 "C16" H 5265 3146 50  0000 L CNN
 F 1 ".01uF" H 5265 3055 50  0000 L CNN
-F 2 "digikey-footprints:0603" H 5188 2950 50  0001 C CNN
+F 2 "smt:C-0603" H 5188 2950 50  0001 C CNN
 F 3 "~" H 5150 3100 50  0001 C CNN
 	1    5150 3100
@@
 F 0 "C8" H 2415 3146 50  0000 L CNN
 F 1 ".01uF" H 2415 3055 50  0000 L CNN
-F 2 "digikey-footprints:0603" H 2338 2950 50  0001 C CNN
+F 2 "smt:C-0603" H 2338 2950 50  0001 C CNN
 F 3 "~" H 2300 3100 50  0001 C CNN
 	1    2300 3100
@@
 F 0 "C6" H 1915 3146 50  0000 L CNN
 F 1 ".01uF" H 1915 3055 50  0000 L CNN
-F 2 "digikey-footprints:0603" H 1838 2950 50  0001 C CNN
+F 2 "smt:C-0603" H 1838 2950 50  0001 C CNN
 F 3 "~" H 1800 3100 50  0001 C CNN
 	1    1800 3100
@@
 F 0 "C15" H 4715 3146 50  0000 L CNN
 F 1 ".01uF" H 4715 3055 50  0000 L CNN
-F 2 "digikey-footprints:0603" H 4638 2950 50  0001 C CNN
+F 2 "smt:C-0603" H 4638 2950 50  0001 C CNN
 F 3 "~" H 4600 3100 50  0001 C CNN
 	1    4600 3100
@@
 F 0 "C13" H 4215 3146 50  0000 L CNN
 F 1 ".01uF" H 4215 3055 50  0000 L CNN
-F 2 "digikey-footprints:0603" H 4138 2950 50  0001 C CNN
+F 2 "smt:C-0603" H 4138 2950 50  0001 C CNN
 F 3 "~" H 4100 3100 50  0001 C CNN
 	1    4100 3100
@@
 F 0 "C12" H 3765 3146 50  0000 L CNN
 F 1 ".01uF" H 3765 3055 50  0000 L CNN
-F 2 "digikey-footprints:0603" H 3688 2950 50  0001 C CNN
+F 2 "smt:C-0603" H 3688 2950 50  0001 C CNN
 F 3 "~" H 3650 3100 50  0001 C CNN
 	1    3650 3100
@@
 F 0 "C10" H 3265 3146 50  0000 L CNN
 F 1 ".01uF" H 3265 3055 50  0000 L CNN
-F 2 "digikey-footprints:0603" H 3188 2950 50  0001 C CNN
+F 2 "smt:C-0603" H 3188 2950 50  0001 C CNN
 F 3 "~" H 3150 3100 50  0001 C CNN
 	1    3150 3100
@@
 F 0 "C9" H 2815 3146 50  0000 L CNN
 F 1 ".01uF" H 2815 3055 50  0000 L CNN
-F 2 "digikey-footprints:0603" H 2738 2950 50  0001 C CNN
+F 2 "smt:C-0603" H 2738 2950 50  0001 C CNN
 F 3 "~" H 2700 3100 50  0001 C CNN
 	1    2700 3100
@@
 F 0 "C29" H 8765 2546 50  0000 L CNN
 F 1 ".01uF" H 8765 2455 50  0000 L CNN
-F 2 "digikey-footprints:0603" H 8688 2350 50  0001 C CNN
+F 2 "smt:C-0603" H 8688 2350 50  0001 C CNN
 F 3 "~" H 8650 2500 50  0001 C CNN
 	1    8650 2500
@@
 F 0 "C27" H 8265 2546 50  0000 L CNN
 F 1 ".01uF" H 8265 2455 50  0000 L CNN
-F 2 "digikey-footprints:0603" H 8188 2350 50  0001 C CNN
+F 2 "smt:C-0603" H 8188 2350 50  0001 C CNN
 F 3 "~" H 8150 2500 50  0001 C CNN
 	1    8150 2500
@@
 F 0 "C26" H 7815 2546 50  0000 L CNN
 F 1 ".01uF" H 7815 2455 50  0000 L CNN
-F 2 "digikey-footprints:0603" H 7738 2350 50  0001 C CNN
+F 2 "smt:C-0603" H 7738 2350 50  0001 C CNN
 F 3 "~" H 7700 2500 50  0001 C CNN
 	1    7700 2500
@@
 F 0 "C25" H 7315 2546 50  0000 L CNN
 F 1 ".01uF" H 7315 2455 50  0000 L CNN
-F 2 "digikey-footprints:0603" H 7238 2350 50  0001 C CNN
+F 2 "smt:C-0603" H 7238 2350 50  0001 C CNN
 F 3 "~" H 7200 2500 50  0001 C CNN
 	1    7200 2500
@@
 F 0 "C23" H 6865 2546 50  0000 L CNN
 F 1 ".01uF" H 6865 2455 50  0000 L CNN
-F 2 "digikey-footprints:0603" H 6788 2350 50  0001 C CNN
+F 2 "smt:C-0603" H 6788 2350 50  0001 C CNN
 F 3 "~" H 6750 2500 50  0001 C CNN
 	1    6750 2500
@@
 F 0 "C21" H 6315 2546 50  0000 L CNN
 F 1 ".01uF" H 6315 2455 50  0000 L CNN
-F 2 "digikey-footprints:0603" H 6238 2350 50  0001 C CNN
+F 2 "smt:C-0603" H 6238 2350 50  0001 C CNN
 F 3 "~" H 6200 2500 50  0001 C CNN
 	1    6200 2500
@@
 F 0 "C19" H 5815 2546 50  0000 L CNN
 F 1 ".01uF" H 5815 2455 50  0000 L CNN
-F 2 "digikey-footprints:0603" H 5738 2350 50  0001 C CNN
+F 2 "smt:C-0603" H 5738 2350 50  0001 C CNN
 F 3 "~" H 5700 2500 50  0001 C CNN
 	1    5700 2500
@@
 	2100 6050 750  6050
 Wire Wire Line
-	7100 7050 7100 7150
-Wire Wire Line
 	7100 5350 7100 5500
 Wire Wire Line
@@
 	1500 5350 2250 5350
 Connection ~ 2250 5350
-Connection ~ 7100 7050
 $Comp
 L dk_Diodes-Zener-Single:1N5231BTR Z2
@@
 F 0 "C31" V 10255 1250 60  0000 C CNB
 F 1 "1uF" V 10350 1250 45  0000 C CNN
-F 2 "digikey-footprints:0603" H 10535 1095 40  0001 L CNN
+F 2 "smt:C-0805" H 10535 1095 40  0001 L CNN
 F 3 "" H 10500 1350 60  0001 C CNN
 F 4 "-" H 10540 1415 45  0001 L CNN "Part"
@@
 F 0 "C30" H 9108 1142 60  0000 L CNB
 F 1 "2.2uF" H 9108 1047 45  0000 L CNN
-F 2 "digikey-footprints:0603" H 9035 945 40  0001 L CNN
+F 2 "smt:C-0805" H 9035 945 40  0001 L CNN
 F 3 "" H 9000 1200 60  0001 C CNN
 F 4 "-" H 9040 1265 45  0001 L CNN "Part"
@@
 F 0 "C28" H 8558 1692 60  0000 L CNB
 F 1 "2.2uF" H 8558 1597 45  0000 L CNN
-F 2 "digikey-footprints:0603" H 8485 1495 40  0001 L CNN
+F 2 "smt:C-0805" H 8485 1495 40  0001 L CNN
 F 3 "" H 8450 1750 60  0001 C CNN
 F 4 "-" H 8490 1815 45  0001 L CNN "Part"
@@
 	10300 5850 8950 5850
 Wire Wire Line
-	15300 6850 15300 6950
-Wire Wire Line
 	15300 5150 15300 5300
 Wire Wire Line
@@
 	9700 5150 10450 5150
 Connection ~ 10450 5150
-Connection ~ 15300 6850
 $Comp
 L dk_Diodes-Zener-Single:1N5231BTR Z7
@@
 F 0 "C44" H 7658 3092 60  0000 L CNB
 F 1 "4.7uF" H 7658 2997 45  0000 L CNN
-F 2 "digikey-footprints:0603" H 7585 2895 40  0001 L CNN
+F 2 "smt:C-0805" H 7585 2895 40  0001 L CNN
 F 3 "" H 7550 3150 60  0001 C CNN
 F 4 "-" H 7590 3215 45  0001 L CNN "Part"

Commit message: the PCB is complete and has been ordered
Parts:
- removed C11: 100uF, digikey-footprints:0805, symbol Device:C
- removed C14, C7: 100nF, smt:C-0603, symbol Device:C
- removed C17: 100uF, digikey-footprints:1206, symbol Device:C
- removed U4: LD1117S33TR_SOT223, TO_SOT_Packages_SMD:SOT-223-3_TabPin2, symbol Regulator_Linear:LD1117S33TR_SOT223
- removed U5: LD1117S50TR_SOT223, TO_SOT_Packages_SMD:SOT-223-3_TabPin2, symbol Regulator_Linear:LD1117S50TR_SOT223
- added C11, C17: 8.2nF, Capacitors_SMD:C_0603_HandSoldering, symbol passive:CAP
- added C14, C7: 22uF, Capacitors_SMD:C_0805_HandSoldering, symbol passive:CAP
- added C50, C52: 100nF, Capacitors_SMD:C_0603_HandSoldering, symbol passive:CAP
- added C51, C53: 47uF, Capacitors_SMD:C_0805_HandSoldering, symbol passive:CAP
- added L8, L9: 3.3uH, digikey-footprints:0805, symbol passive:INDUCTOR
- added R60, R64: 100K, Resistor_SMD:R_0402_1005Metric, symbol passive:RESISTOR
- added R61: 56.2K, Resistor_SMD:R_0402_1005Metric, symbol passive:RESISTOR
- added R62, R66: 10K, Resistor_SMD:R_0402_1005Metric, symbol passive:RESISTOR
- added R65: 33.2K, Resistor_SMD:R_0402_1005Metric, symbol passive:RESISTOR
- added U4, U5: TPS563210, TO_SOT_Packages_SMD:SOT-23-8_Handsoldering, symbol dk_PMIC-Voltage-Regulators-DC-DC-Switching-Regulators:TPS563210
Connections:
- wire segments 240 -> 279

Commit message: CLEANED UP THE SCHEMATICS ADDED NEADED FIXES FOUND ON THE BOARD
Other:
- note added: "-3V3 SWITCHING SUPPLY"
- note added: "3V3 SWITCHING SUPPLY"
- note added: "5V SWITCHING SUPPLY"
- note added: "RECHECK THE NUMBER OF DECOUPLING CAPS"
- note added: "THE HOLE SIZES NEED TO BE CHANGED THE FOOTPRINT IS BAD"
- note added: "THESE PORTS SHOULD BE REMAPED, THE GARMIN SHOULD BE CONTROLLED DIFFERENTLY THAN PWR"
- note added: "WE SHOULD ADD A -5V SUPPLY and a 3way switch"
Changed lines of the file:
@@
 U 1 1 5B982AEC
 P 10500 1250
-F 0 "C31" V 10255 1250 60  0000 C CNB
-F 1 "1uF" V 10350 1250 45  0000 C CNN
+F 0 "C31" V 10550 1400 60  0000 C CNB
+F 1 "1uF" V 10650 1400 45  0000 C CNN
 F 2 "smt:C-0805" H 10535 1095 40  0001 L CNN
 F 3 "" H 10500 1350 60  0001 C CNN
@@
 U 1 1 5B9C3F0C
 P 9000 1100
-F 0 "C30" H 9108 1142 60  0000 L CNB
-F 1 "2.2uF" H 9108 1047 45  0000 L CNN
+F 0 "C30" H 8750 1200 60  0000 L CNB
+F 1 "2.2uF" H 8750 1050 45  0000 L CNN
 F 2 "smt:C-0805" H 9035 945 40  0001 L CNN
 F 3 "" H 9000 1200 60  0001 C CNN
@@
 	9000 950  9000 1000
 Connection ~ 9000 950
-Wire Wire Line
-	9000 950  8650 950
 Wire Wire Line
 	9000 1200 9000 1250
@@
 P 10250 1400
 F 0 "#PWR052" H 10250 1250 50  0001 C CNN
-F 1 "+3V3" H 10265 1573 50  0000 C CNN
+F 1 "+3V3" H 10350 1500 50  0000 C CNN
 F 2 "" H 10250 1400 50  0001 C CNN
 F 3 "" H 10250 1400 50  0001 C CNN
@@
 L power:-3V3 #PWR045
 U 1 1 5BB79549
-P 8650 950
-F 0 "#PWR045" H 8650 1050 50  0001 C CNN
-F 1 "-3V3" H 8665 1123 50  0000 C CNN
-F 2 "" H 8650 950 50  0001 C CNN
-F 3 "" H 8650 950 50  0001 C CNN
-	1    8650 950
+P 8550 950
+F 0 "#PWR045" H 8550 1050 50  0001 C CNN
+F 1 "-3V3" H 8565 1123 50  0000 C CNN
+F 2 "" H 8550 950 50  0001 C CNN
+F 3 "" H 8550 950 50  0001 C CNN
+	1    8550 950
 	-1   0    0    1
 $EndComp
@@
 Wire Wire Line
 	4450 1950 4500 1950
+Text Notes 8550 7700 0    50   ~ 0
+THESE PORTS SHOULD BE REMAPED, THE GARMIN SHOULD BE CONTROLLED DIFFERENTLY THAN PWR
+Text Notes 2100 1650 0    50   ~ 0
+5V SWITCHING SUPPLY
+Text Notes 4900 3700 0    50   ~ 0
+3V3 SWITCHING SUPPLY
+Text Notes 8350 750  0    50   ~ 0
+-3V3 SWITCHING SUPPLY
+Text Notes 8000 3050 0    50   ~ 0
+RECHECK THE NUMBER OF DECOUPLING CAPS
+Text Notes 5200 2050 0    50   ~ 0
+WE SHOULD ADD A -5V SUPPLY and a 3way switch
+Text Notes 1350 1250 0    50   ~ 0
+THE HOLE SIZES NEED TO BE CHANGED THE FOOTPRINT IS BAD
+Wire Wire Line
+	8550 950  9000 950
 $EndSCHEMATC

Commit message: USB test instrument support and SCPI support were added to the FW
Parts:
- U4, U5: symbol dk_PMIC-Voltage-Regulators-DC-DC-Switching-Regulators:TPS563210 -> SchematicAutomation-cache:TPS563210
- U6: symbol Power_Management:LM2776 -> NegativeRail:LM2776
Connections:
- wire segments 279 -> 283
Changed lines of the file:
@@
 $EndComp
 Wire Wire Line
-	1250 1100 1600 1100
+	1250 1100 1550 1100
 $Comp
 L power:+12V #PWR?
@@
 $EndComp
 Wire Wire Line
-	6300 750  6950 750
+	6300 750  6800 750
 $Comp
 L dk_Toggle-Switches:ATE1D-2M3-10-Z S2
@@
 	7500 1800 7300 1800
 Wire Wire Line
-	6250 1350 6900 1350
+	6250 1350 6650 1350
 Wire Wire Line
 	7800 1600 7800 1700
@@
 $EndComp
 $Comp
-L Power_Management:LM2776 U6
+L NegativeRail:LM2776 U6
 U 1 1 5B9767C0
 P 9700 1050
@@
 	10450 5950 10450 5850
 $Comp
-L dk_PMIC-Voltage-Regulators-DC-DC-Switching-Regulators:TPS563210 U4
+L SchematicAutomation-cache:TPS563210 U4
 U 1 1 5B983547
-P 2250 1800
-F 0 "U4" H 2250 1915 50  0000 C CNN
-F 1 "TPS563210" H 2250 1824 50  0000 C CNN
-F 2 "TO_SOT_Packages_SMD:SOT-23-8_Handsoldering" H 2250 1800 50  0001 C CNN
-F 3 "http://www.ti.com/lit/ds/symlink/tps563210.pdf" H 2250 1800 50  0001 C CNN
-	1    2250 1800
+P 2300 1750
+F 0 "U4" H 2300 1865 50  0000 C CNN
+F 1 "TPS563210" H 2300 1774 50  0000 C CNN
+F 2 "TO_SOT_Packages_SMD:SOT-23-8_Handsoldering" H 2300 1750 50  0001 C CNN
+F 3 "http://www.ti.com/lit/ds/symlink/tps563210.pdf" H 2300 1750 50  0001 C CNN
+	1    2300 1750
 	1    0    0    -1
 $EndComp
@@
 	1550 1950 850  1950
 $Comp
-L dk_PMIC-Voltage-Regulators-DC-DC-Switching-Regulators:TPS563210 U5
+L SchematicAutomation-cache:TPS563210 U5
 U 1 1 5BB6AF17
-P 2700 3700
-F 0 "U5" H 2700 3815 50  0000 C CNN
-F 1 "TPS563210" H 2700 3724 50  0000 C CNN
-F 2 "TO_SOT_Packages_SMD:SOT-23-8_Handsoldering" H 2700 3700 50  0001 C CNN
-F 3 "http://www.ti.com/lit/ds/symlink/tps563210.pdf" H 2700 3700 50  0001 C CNN
-	1    2700 3700
+P 2750 3650
+F 0 "U5" H 2750 3765 50  0000 C CNN
+F 1 "TPS563210" H 2750 3674 50  0000 C CNN
+F 2 "TO_SOT_Packages_SMD:SOT-23-8_Handsoldering" H 2750 3650 50  0001 C CNN
+F 3 "http://www.ti.com/lit/ds/symlink/tps563210.pdf" H 2750 3650 50  0001 C CNN
+	1    2750 3650
 	1    0    0    -1
 $EndComp
@@
 	3150 4100 3950 4100
 Wire Wire Line
-	4250 3850 4550 3850
+	4250 3850 4300 3850
 Connection ~ 4250 3850
 Wire Wire Line
@@
 Wire Wire Line
 	8550 950  9000 950
+$Comp
+L power:PWR_FLAG #FLG0109
+U 1 1 5BC6592E
+P 1550 1100
+F 0 "#FLG0109" H 1550 1175 50  0001 C CNN
+F 1 "PWR_FLAG" H 1550 1274 50  0000 C CNN
+F 2 "" H 1550 1100 50  0001 C CNN
+F 3 "~" H 1550 1100 50  0001 C CNN
+	1    1550 1100
+	1    0    0    -1
+$EndComp
+Connection ~ 1550 1100
+Wire Wire Line
+	1550 1100 1600 1100
+$Comp
+L power:PWR_FLAG #FLG0110
+U 1 1 5BC65EE9
+P 6800 750
+F 0 "#FLG0110" H 6800 825 50  0001 C CNN
+F 1 "PWR_FLAG" H 6800 924 50  0000 C CNN
+F 2 "" H 6800 750 50  0001 C CNN
+F 3 "~" H 6800 750 50  0001 C CNN
+	1    6800 750
+	1    0    0    -1
+$EndComp
+Connection ~ 6800 750
+Wire Wire Line
+	6800 750  6950 750
+$Comp
+L power:PWR_FLAG #FLG0111
+U 1 1 5BC65F97
+P 6650 1350
+F 0 "#FLG0111" H 6650 1425 50  0001 C CNN
+F 1 "PWR_FLAG" H 6650 1524 50  0000 C CNN
+F 2 "" H 6650 1350 50  0001 C CNN
+F 3 "~" H 6650 1350 50  0001 C CNN
+	1    6650 1350
+	1    0    0    -1
+$EndComp
+Connection ~ 6650 1350
+Wire Wire Line
+	6650 1350 6900 1350
+$Comp
+L power:PWR_FLAG #FLG0112
+U 1 1 5BC66942
+P 4300 3850
+F 0 "#FLG0112" H 4300 3925 50  0001 C CNN
+F 1 "PWR_FLAG" H 4300 4024 50  0000 C CNN
+F 2 "" H 4300 3850 50  0001 C CNN
+F 3 "~" H 4300 3850 50  0001 C CNN
+	1    4300 3850
+	1    0    0    -1
+$EndComp
+Connection ~ 4300 3850
+Wire Wire Line
+	4300 3850 4550 3850
 $EndSCHEMATC
