File: QualificationTestingAutomation/SchematicAutomation/UART.sch (KiCad schematic (older format))
At the start: 21 parts, among them Q3 2N7002DW, Q4 2N7002DW, Q5 2N7002DW, Q6 2N7002DW, U20 CD4070B

Commit message: C WPCB was started and the schematic is full, I am thinking of implementing the UART test using analog muxes.
Parts:
- removed R19, R20, R21, R22, R23, R24, R25, R26: 10k, digikey-footprints:0603, symbol passive:RESISTOR
- R11, R12, R13, R14, R15, R16, R17, R18: footprint digikey-footprints:0603 -> Resistor_SMD:R_0402_1005Metric
Connections:
- wire segments 87 -> 76

Commit message: the PCB is complete and has been ordered
Parts:
- added U32: MAX324CUA, Housings_SSOP:MSOP-8_3x3mm_Pitch0.65mm, symbol Analog_Switch:MAX324CUA
Connections:
- net labels added: CTS_CONT, TX_CONT
- net labels removed: +5V
- wire segments 76 -> 78

Commit message: Basis for the software
Parts:
- added R? (x6): 10k, Resistor_SMD:R_0402_1005Metric, symbol passive:RESISTOR
Connections:
- wire segments 78 -> 85
