File: QualificationTestingAutomation/SchematicAutomation/UART.sch (KiCad schematic (older format))
At the start: 14 parts, among them Q3 2N7002DW, Q4 2N7002DW, Q5 2N7002DW, Q6 2N7002DW, U20 CD4070B, U32 MAX324CUA

Commit message: CLEANED UP THE SCHEMATICS ADDED NEADED FIXES FOUND ON THE BOARD
Parts:
- added R? (x2): R0, symbol passive:RESISTOR
- added R? (x2): 100k, Resistor_SMD:R_0402_1005Metric, symbol passive:RESISTOR
- added R? (x2): 56K, symbol passive:RESISTOR
- added R?: RESISTOR, symbol passive:RESISTOR
Connections:
- wire segments 78 -> 106
Other:
- note added: "BYPASS RESISTORS"
- note added: "SHOULD WE ADD BIASING RESISTORS JUST IN CASE"
- note added: "THESE SHORTS are to bypass the switch"
- note added: "THIS MUX will be kept but not populated"
- note added: "WE SHOULD ADD MORE DECOUPLING CAPS"

Commit message: USB test instrument support and SCPI support were added to the FW
Parts:
- U20: symbol dk_Interface-Drivers-Receivers-Transceivers:CD4070B -> 4XXXSeriesLOGIC:CD4070B
- gave numbers to parts that had none: 7

Commit message: RX TX mixup was solved by changing RX_3V3 and TX_3V3 on the XOR side Same goes for CTS and RTS and some general clean up
Signed-off-by: Riyad Alalami <riyadhelalami@gmail.com>
Changed lines of the file:
@@
 $Descr A4 11693 8268
 encoding utf-8
-Sheet 15 16
+Sheet 8 16
 Title ""
 Date ""
@@
 AR Path="/5BB9E3C7/5BDC515F/5C46C79B" Ref="#PWR0253"  Part="1"
 AR Path="/5BB9E3C7/5BDC5169/5C46C79B" Ref="#PWR0272"  Part="1"
-F 0 "#PWR0253" H 2150 4050 50  0001 C CNN
+F 0 "#PWR0101" H 2150 4050 50  0001 C CNN
 F 1 "GND" H 2155 4127 50  0000 C CNN
 F 2 "" H 2150 4300 50  0001 C CNN
@@
 AR Path="/5BB9E3C7/5BDC515F/5C46C7A1" Ref="#PWR0258"  Part="1"
 AR Path="/5BB9E3C7/5BDC5169/5C46C7A1" Ref="#PWR0277"  Part="1"
-F 0 "#PWR0258" H 4750 4700 50  0001 C CNN
+F 0 "#PWR0106" H 4750 4700 50  0001 C CNN
 F 1 "GND" H 4755 4777 50  0000 C CNN
 F 2 "" H 4750 4950 50  0001 C CNN
@@
 AR Path="/5BB9E3C7/5BDC515F/5C46C7C8" Ref="#PWR0261"  Part="1"
 AR Path="/5BB9E3C7/5BDC5169/5C46C7C8" Ref="#PWR0280"  Part="1"
-F 0 "#PWR0261" H 5550 3400 50  0001 C CNN
+F 0 "#PWR0109" H 5550 3400 50  0001 C CNN
 F 1 "GND" H 5555 3477 50  0000 C CNN
 F 2 "" H 5550 3650 50  0001 C CNN
@@
 AR Path="/5BB9E3C7/5BDC515F/5C46C897" Ref="#PWR0262"  Part="1"
 AR Path="/5BB9E3C7/5BDC5169/5C46C897" Ref="#PWR0281"  Part="1"
-F 0 "#PWR0262" H 6850 3400 50  0001 C CNN
+F 0 "#PWR0110" H 6850 3400 50  0001 C CNN
 F 1 "GND" H 6855 3477 50  0000 C CNN
 F 2 "" H 6850 3650 50  0001 C CNN
@@
 Text HLabel 5500 4600 2    50   Input ~ 0
 TX
+Text HLabel 5900 2750 0    50   Input ~ 0
+Tx_3V3
 Text HLabel 5650 3300 0    50   Input ~ 0
-Tx_3V3
-Text HLabel 5900 2750 0    50   Input ~ 0
 RX_3V3
-Text HLabel 6550 2750 2    50   Input ~ 0
+Text HLabel 6500 3300 2    50   Input ~ 0
 RTS_3V3
 Wire Wire Line
@@
 AR Path="/5BB9E3C7/5BDC515F/5BBDD3AA" Ref="#PWR0263"  Part="1"
 AR Path="/5BB9E3C7/5BDC5169/5BBDD3AA" Ref="#PWR0282"  Part="1"
-F 0 "#PWR0263" H 7000 2400 50  0001 C CNN
+F 0 "#PWR0111" H 7000 2400 50  0001 C CNN
 F 1 "+3V3" H 7015 2723 50  0000 C CNN
 F 2 "" H 7000 2550 50  0001 C CNN
@@
 AR Path="/5BB9E3C7/5BDC515F/5BC06776" Ref="#PWR0255"  Part="1"
 AR Path="/5BB9E3C7/5BDC5169/5BC06776" Ref="#PWR0274"  Part="1"
-F 0 "#PWR0255" H 4800 2200 50  0001 C CNN
+F 0 "#PWR0103" H 4800 2200 50  0001 C CNN
 F 1 "+VSW" H 4815 2523 50  0000 C CNN
 F 2 "" H 4800 2350 50  0001 C CNN
@@
 AR Path="/5BB9E3C7/5BDC515F/5BC0F576" Ref="#PWR0256"  Part="1"
 AR Path="/5BB9E3C7/5BDC5169/5BC0F576" Ref="#PWR0275"  Part="1"
-F 0 "#PWR0256" H 2200 2550 50  0001 C CNN
+F 0 "#PWR0104" H 2200 2550 50  0001 C CNN
 F 1 "-VSW" H 2215 2623 50  0000 C CNN
 F 2 "" H 2200 2450 50  0001 C CNN
@@
 AR Path="/5BB9E3C7/5BDC515F/5BC1421C" Ref="#PWR0259"  Part="1"
 AR Path="/5BB9E3C7/5BDC5169/5BC1421C" Ref="#PWR0278"  Part="1"
-F 0 "#PWR0259" H 10650 3950 50  0001 C CNN
+F 0 "#PWR0107" H 10650 3950 50  0001 C CNN
 F 1 "GND" H 10655 4027 50  0000 C CNN
 F 2 "" H 10650 4200 50  0001 C CNN
@@
 AR Path="/5BB9E3C7/5BDC515F/5BC14222" Ref="#PWR0260"  Part="1"
 AR Path="/5BB9E3C7/5BDC5169/5BC14222" Ref="#PWR0279"  Part="1"
-F 0 "#PWR0260" H 8050 4600 50  0001 C CNN
+F 0 "#PWR0108" H 8050 4600 50  0001 C CNN
 F 1 "GND" H 8055 4677 50  0000 C CNN
 F 2 "" H 8050 4850 50  0001 C CNN
@@
 AR Path="/5BB9E3C7/5BDC515F/5BC1427E" Ref="#PWR0266"  Part="1"
 AR Path="/5BB9E3C7/5BDC5169/5BC1427E" Ref="#PWR0285"  Part="1"
-F 0 "#PWR0266" H 8000 2100 50  0001 C CNN
+F 0 "#PWR0114" H 8000 2100 50  0001 C CNN
 F 1 "+VSW" H 8015 2423 50  0000 C CNN
 F 2 "" H 8000 2250 50  0001 C CNN
@@
 AR Path="/5BB9E3C7/5BDC515F/5BC14284" Ref="#PWR0267"  Part="1"
 AR Path="/5BB9E3C7/5BDC5169/5BC14284" Ref="#PWR0286"  Part="1"
-F 0 "#PWR0267" H 10600 2450 50  0001 C CNN
+F 0 "#PWR0115" H 10600 2450 50  0001 C CNN
 F 1 "-VSW" H 10615 2523 50  0000 C CNN
 F 2 "" H 10600 2350 50  0001 C CNN
@@
 AR Path="/5BB9E3C7/5BDC515F/5BC1C74A" Ref="#PWR0268"  Part="1"
 AR Path="/5BB9E3C7/5BDC5169/5BC1C74A" Ref="#PWR0287"  Part="1"
-F 0 "#PWR0268" H 4800 3200 50  0001 C CNN
+F 0 "#PWR0116" H 4800 3200 50  0001 C CNN
 F 1 "-VSW" H 4815 3273 50  0000 C CNN
 F 2 "" H 4800 3100 50  0001 C CNN
@@
 AR Path="/5BB9E3C7/5BDC515F/5BC1F98F" Ref="#PWR0269"  Part="1"
 AR Path="/5BB9E3C7/5BDC5169/5BC1F98F" Ref="#PWR0288"  Part="1"
-F 0 "#PWR0269" H 2200 2800 50  0001 C CNN
+F 0 "#PWR0117" H 2200 2800 50  0001 C CNN
 F 1 "+VSW" H 2215 3123 50  0000 C CNN
 F 2 "" H 2200 2950 50  0001 C CNN
@@
 AR Path="/5BB9E3C7/5BDC515F/5BC24646" Ref="#PWR0270"  Part="1"
 AR Path="/5BB9E3C7/5BDC5169/5BC24646" Ref="#PWR0289"  Part="1"
-F 0 "#PWR0270" H 8000 3100 50  0001 C CNN
+F 0 "#PWR0118" H 8000 3100 50  0001 C CNN
 F 1 "-VSW" H 8015 3173 50  0000 C CNN
 F 2 "" H 8000 3000 50  0001 C CNN
@@
 AR Path="/5BB9E3C7/5BDC515F/5BC26035" Ref="#PWR0271"  Part="1"
 AR Path="/5BB9E3C7/5BDC5169/5BC26035" Ref="#PWR0290"  Part="1"
-F 0 "#PWR0271" H 10600 2750 50  0001 C CNN
+F 0 "#PWR0119" H 10600 2750 50  0001 C CNN
 F 1 "+VSW" H 10615 3073 50  0000 C CNN
 F 2 "" H 10600 2900 50  0001 C CNN
@@
 	1    0    0    -1
 $EndComp
-Text HLabel 6500 3300 2    50   Input ~ 0
+Text HLabel 6550 2750 2    50   Input ~ 0
 CTS_3V3
 $Comp
@@
 AR Path="/5BB9E3C7/5BDC515F/5BD72BE1" Ref="#PWR0248"  Part="1"
 AR Path="/5BB9E3C7/5BDC5169/5BD72BE1" Ref="#PWR?"  Part="1"
-F 0 "#PWR0248" H 6000 5050 50  0001 C CNN
+F 0 "#PWR0234" H 6000 5050 50  0001 C CNN
 F 1 "-VSW" H 6015 5123 50  0000 C CNN
 F 2 "" H 6000 4950 50  0001 C CNN
@@
 AR Path="/5BB9E3C7/5BDC515F/5BD81C4F" Ref="#PWR0249"  Part="1"
 AR Path="/5BB9E3C7/5BDC5169/5BD81C4F" Ref="#PWR?"  Part="1"
-F 0 "#PWR0249" H 7000 4800 50  0001 C CNN
+F 0 "#PWR0235" H 7000 4800 50  0001 C CNN
 F 1 "+VSW" H 7015 5123 50  0000 C CNN
 F 2 "" H 7000 4950 50  0001 C CNN
@@
 AR Path="/5BB9E3C7/5BD54793/5BE5B408" Ref="#PWR0188"  Part="1"
 AR Path="/5BB9E3C7/5BDC515F/5BE5B408" Ref="#PWR0200"  Part="1"
-F 0 "#PWR0200" H 4750 4100 50  0001 C CNN
+F 0 "#PWR0102" H 4750 4100 50  0001 C CNN
 F 1 "+3V3" H 4765 4423 50  0000 C CNN
 F 2 "" H 4750 4250 50  0001 C CNN
@@
 AR Path="/5BB9E3C7/5BD54793/5BE5B5DF" Ref="#PWR0189"  Part="1"
 AR Path="/5BB9E3C7/5BDC515F/5BE5B5DF" Ref="#PWR0207"  Part="1"
-F 0 "#PWR0207" H 10650 4550 50  0001 C CNN
+F 0 "#PWR0105" H 10650 4550 50  0001 C CNN
 F 1 "+3V3" H 10665 4873 50  0000 C CNN
 F 2 "" H 10650 4700 50  0001 C CNN
@@
 AR Path="/5BB9E3C7/5BD54793/5BE69AE3" Ref="#PWR0197"  Part="1"
 AR Path="/5BB9E3C7/5BDC515F/5BE69AE3" Ref="#PWR0208"  Part="1"
-F 0 "#PWR0208" H 2100 4650 50  0001 C CNN
+F 0 "#PWR0112" H 2100 4650 50  0001 C CNN
 F 1 "+3V3" H 2115 4973 50  0000 C CNN
 F 2 "" H 2100 4800 50  0001 C CNN
@@
 AR Path="/5BB9E3C7/5BD54793/5BE6B6A9" Ref="#PWR0274"  Part="1"
 AR Path="/5BB9E3C7/5BDC515F/5BE6B6A9" Ref="#PWR0275"  Part="1"
-F 0 "#PWR0275" H 8050 4000 50  0001 C CNN
+F 0 "#PWR0254" H 8050 4000 50  0001 C CNN
 F 1 "+3V3" H 8065 4323 50  0000 C CNN
 F 2 "" H 8050 4150 50  0001 C CNN
