File: QualificationTestingAutomation/SchematicAutomation/MUXing-2.sch (KiCad schematic (older format))
At the start: 7 parts, among them U16 MAX14752, U17 MAX14752, U18 MAX14752, U19 MAX14752, U20 MAX14752, U21 MAX14752, U22 MAX14752

Commit message: schematic is finished a few symbols were added, footprints are almost done, some work needs to be done on the connectors#
Parts:
- added J17: BananaPlug, symbol Connector_Generic:Conn_01x02
- added U1, U16, U2: DG408LE, digikey-footprints:TSSOP-16-1EP_W4.40mm, symbol Analog_Switch:DG408LE
- added U17: DS18B20_, digikey-footprints:TO-92-3, symbol dk_Temperature-Sensors-Analog-and-Digital-Output:DS18B20_
- added U19: CD74HC4067SM96, digikey-footprints:SSOP-24_W5.30mm, symbol dk_Interface-Analog-Switches-Multiplexers-Demultiplexers:CD74HC4067SM96
- renumbered U19 to U10, U20 to U11, U21 to U12, U22 to U13, U16 to U7, U17 to U8, U18 to U9
Connections:
- net labels added: +5V, 1_OUT0, 1_OUT1, 1_OUT2, 1_OUT3, 1_OWB_MAIN, 1_OWB_SEC, 2_OUT0, 2_OUT1, 2_OUT2, 2_OUT3, 2_OWB_MAIN, 2_OWB_SEC, 3_OUT0, 3_OUT1, 3_OUT2, 3_OUT3, 3_OWB_MAIN, 3_OWB_SEC, 4_OUT0, 4_OUT1, 4_OUT2, 4_OUT3, 4_OWB_MAIN, 4_OWB_SEC, 5_OUT0, 5_OUT1, 5_OUT2, 5_OUT3, 5_OWB_MAIN, 5_OWB_SEC, MUX24, MUX25, MUX26, MUXA1
- wire segments 124 -> 231
- no-connect marks 0 -> 17

Commit message: C WPCB was started and the schematic is full, I am thinking of implementing the UART test using analog muxes.
Parts:
- J17: value BananaPlug -> Banana Jack; footprint (none) -> Connectors:Banana_Jack_2Pin; Description (none) -> The hole has a diameter of about 5.2mm (fits standard 4mm b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
- U1, U16: footprint digikey-footprints:TSSOP-16-1EP_W4.40mm -> digikey-footprints:SOIC-16_W3.90mm; Digi-Key_PN (none) -> DG408LEDY-T1-GE3CT-ND; MPN (none) -> DG408LEDY-T1-GE3
- U10, U11, U12, U13, U7, U8, U9: Digi-Key_PN (none) -> MAX14752EUE+-ND
- U2: footprint digikey-footprints:TSSOP-16-1EP_W4.40mm -> digikey-footprints:SOIC-16_W3.90mm; Digi-Key_PN (none) -> DG408LEDY-T1-GE3CT-ND; MPN (none) -> DG408LEDY-T1-GE3; PN DG408LEDQ-T1-GE3CT-ND -> (none)
Connections:
- wire segments 231 -> 228
Changed lines of the file:
@@
 $Descr B 17000 11000
 encoding utf-8
-Sheet 6 18
+Sheet 6 16
 Title ""
 Date ""
@@
 F 1 "MAX14752" H 2125 1724 50  0000 C CNN
 F 2 "digikey-footprints:TSSOP-16-1EP_W4.40mm" H 2150 1800 50  0001 C CNN
-F 3 "" H 2150 1800 50  0001 C CNN
+F 3 "https://datasheets.maximintegrated.com/en/ds/MAX14752-MAX14753.pdf" H 2150 1800 50  0001 C CNN
+F 4 " MAX14752EUE+-ND " H 0   0   50  0001 C CNN "Digi-Key_PN"
 	1    2100 1700
 	1    0    0    -1
@@
 F 1 "MAX14752" H 4125 1674 50  0000 C CNN
 F 2 "digikey-footprints:TSSOP-16-1EP_W4.40mm" H 4150 1750 50  0001 C CNN
-F 3 "" H 4150 1750 50  0001 C CNN
+F 3 "https://datasheets.maximintegrated.com/en/ds/MAX14752-MAX14753.pdf" H 4150 1750 50  0001 C CNN
+F 4 " MAX14752EUE+-ND " H 0   0   50  0001 C CNN "Digi-Key_PN"
 	1    4100 1650
 	1    0    0    -1
@@
 F 1 "MAX14752" H 6225 1674 50  0000 C CNN
 F 2 "digikey-footprints:TSSOP-16-1EP_W4.40mm" H 6250 1750 50  0001 C CNN
-F 3 "" H 6250 1750 50  0001 C CNN
+F 3 "https://datasheets.maximintegrated.com/en/ds/MAX14752-MAX14753.pdf" H 6250 1750 50  0001 C CNN
+F 4 " MAX14752EUE+-ND " H 0   0   50  0001 C CNN "Digi-Key_PN"
 	1    6200 1650
 	1    0    0    -1
@@
 F 1 "MAX14752" H 1775 4524 50  0000 C CNN
 F 2 "digikey-footprints:TSSOP-16-1EP_W4.40mm" H 1800 4600 50  0001 C CNN
-F 3 "" H 1800 4600 50  0001 C CNN
+F 3 "https://datasheets.maximintegrated.com/en/ds/MAX14752-MAX14753.pdf" H 1800 4600 50  0001 C CNN
+F 4 " MAX14752EUE+-ND " H 0   0   50  0001 C CNN "Digi-Key_PN"
 	1    1750 4500
 	1    0    0    -1
@@
 F 1 "MAX14752" H 3575 4474 50  0000 C CNN
 F 2 "digikey-footprints:TSSOP-16-1EP_W4.40mm" H 3600 4550 50  0001 C CNN
-F 3 "" H 3600 4550 50  0001 C CNN
+F 3 "https://datasheets.maximintegrated.com/en/ds/MAX14752-MAX14753.pdf" H 3600 4550 50  0001 C CNN
+F 4 " MAX14752EUE+-ND " H 0   0   50  0001 C CNN "Digi-Key_PN"
 	1    3550 4450
 	1    0    0    -1
@@
 F 1 "MAX14752" H 5375 4424 50  0000 C CNN
 F 2 "digikey-footprints:TSSOP-16-1EP_W4.40mm" H 5400 4500 50  0001 C CNN
-F 3 "" H 5400 4500 50  0001 C CNN
+F 3 "https://datasheets.maximintegrated.com/en/ds/MAX14752-MAX14753.pdf" H 5400 4500 50  0001 C CNN
+F 4 " MAX14752EUE+-ND " H 0   0   50  0001 C CNN "Digi-Key_PN"
 	1    5350 4400
 	1    0    0    -1
@@
 F 1 "MAX14752" H 7075 4424 50  0000 C CNN
 F 2 "digikey-footprints:TSSOP-16-1EP_W4.40mm" H 7100 4500 50  0001 C CNN
-F 3 "" H 7100 4500 50  0001 C CNN
+F 3 "https://datasheets.maximintegrated.com/en/ds/MAX14752-MAX14753.pdf" H 7100 4500 50  0001 C CNN
+F 4 " MAX14752EUE+-ND " H 7050 4400 50  0001 C CNN "Digi-Key_PN"
 	1    7050 4400
 	1    0    0    -1
@@
 U 1 1 5BA76687
 P 11100 2100
-F 0 "U2" H 11100 2650 50  0000 C CNN
-F 1 "DG408LE" H 11100 2600 50  0000 C CNN
-F 2 "digikey-footprints:TSSOP-16-1EP_W4.40mm" H 11100 2100 50  0001 C CNN
+F 0 "U2" H 11100 2465 50  0000 C CNN
+F 1 "DG408LE" H 11100 2374 50  0000 C CNN
+F 2 "digikey-footprints:SOIC-16_W3.90mm" H 11100 2100 50  0001 C CNN
 F 3 "http://www.vishay.com/docs/78084/dg408le.pdf" H 11100 2100 50  0001 C CNN
-F 4 "DG408LEDQ-T1-GE3CT-ND " H 11100 2100 50  0001 C CNN "PN"
+F 4 "DG408LEDY-T1-GE3CT-ND " H 11100 2100 50  0001 C CNN "Digi-Key_PN"
+F 5 "DG408LEDY-T1-GE3" H 0   0   50  0001 C CNN "MPN"
 	1    11100 2100
 	1    0    0    -1
@@
 U 1 1 5BB6FE9D
 P 9650 4200
-F 0 "U1" H 9650 4750 50  0000 C CNN
-F 1 "DG408LE" H 9650 4700 50  0000 C CNN
-F 2 "digikey-footprints:TSSOP-16-1EP_W4.40mm" H 9650 4200 50  0001 C CNN
-F 3 "" H 9650 4200 50  0001 C CNN
+F 0 "U1" H 9650 4550 50  0000 C CNN
+F 1 "DG408LE" H 9650 4450 50  0000 C CNN
+F 2 "digikey-footprints:SOIC-16_W3.90mm" H 9650 4200 50  0001 C CNN
+F 3 "http://www.vishay.com/docs/78084/dg408le.pdf" H 9650 4200 50  0001 C CNN
+F 4 "DG408LEDY-T1-GE3CT-ND " H 0   0   50  0001 C CNN "Digi-Key_PN"
+F 5 "DG408LEDY-T1-GE3" H 0   0   50  0001 C CNN "MPN"
 	1    9650 4200
 	1    0    0    -1
@@
 U 1 1 5BB7C29C
 P 11600 4200
-F 0 "U16" H 11600 4750 50  0000 C CNN
-F 1 "DG408LE" H 11600 4700 50  0000 C CNN
-F 2 "digikey-footprints:TSSOP-16-1EP_W4.40mm" H 11600 4200 50  0001 C CNN
-F 3 "" H 11600 4200 50  0001 C CNN
+F 0 "U16" H 11600 4550 50  0000 C CNN
+F 1 "DG408LE" H 11600 4450 50  0000 C CNN
+F 2 "digikey-footprints:SOIC-16_W3.90mm" H 11600 4200 50  0001 C CNN
+F 3 "http://www.vishay.com/docs/78084/dg408le.pdf" H 11600 4200 50  0001 C CNN
+F 4 "DG408LEDY-T1-GE3CT-ND " H 0   0   50  0001 C CNN "Digi-Key_PN"
+F 5 "DG408LEDY-T1-GE3" H 0   0   50  0001 C CNN "MPN"
 	1    11600 4200
 	1    0    0    -1
@@
 	-1   0    0    1
 $EndComp
-Wire Wire Line
-	12600 1450 12800 1450
-Wire Wire Line
-	12800 1750 12800 1450
-Connection ~ 12800 1450
 $Comp
 L power:GND #PWR?
@@
 	1    0    0    -1
 $EndComp
-Wire Wire Line
-	12800 1450 14700 1450
 $Comp
 L dk_Interface-Analog-Switches-Multiplexers-Demultiplexers:CD74HC4067SM96 U?
@@
 Wire Wire Line
 	15200 1150 15700 1150
-Text GLabel 15850 1950 2    50   Input ~ 0
+Text GLabel 15850 1750 2    50   Input ~ 0
 MUXC
 Text GLabel 15850 1850 2    50   Input ~ 0
 MUXD
-Text GLabel 15850 1750 2    50   Input ~ 0
+Text GLabel 15850 1950 2    50   Input ~ 0
 MUXE
 Wire Wire Line
@@
 AR Path="/5BCA1CB6/5BD017D0" Ref="J17"  Part="1"
 F 0 "J17" H 9980 5792 50  0000 L CNN
-F 1 "BananaPlug" H 9980 5701 50  0000 L CNN
-F 2 "" H 9900 5800 50  0001 C CNN
+F 1 "Banana Jack" H 9980 5701 50  0000 L CNN
+F 2 "Connectors:Banana_Jack_2Pin" H 9900 5800 50  0001 C CNN
 F 3 "~" H 9900 5800 50  0001 C CNN
 F 4 "Multimeter" H 9900 5800 50  0001 C CNN "Field4"
+F 5 "The hole has a diameter of about 5.2mm (fits standard 4mm banana plugs), the cap on the front has an outside diameter of about 11.6mm and length of 15.2mm. Diameter of the screw is 3.8mm. The mounting key is about 4 x 5.4mm." H 0   0   50  0001 C CNN "Description"
 	1    9900 5800
 	1    0    0    -1
@@
 	-1   0    0    1
 $EndComp
-Connection ~ 12700 1750
-Wire Wire Line
-	12700 1750 12800 1750
+Wire Wire Line
+	12600 1450 14700 1450
 $EndSCHEMATC

Commit message: CLEANED UP THE SCHEMATICS ADDED NEADED FIXES FOUND ON THE BOARD
Connections:
- wire segments 228 -> 226
Other:
- note added: "IN/ADC MULTIPLEXING"
- note added: "OUTPUT MULTIPLEXING"
- note added: "OWB MULTIPLEXING"
Changed lines of the file:
@@
 Wire Wire Line
 	3750 2800 3500 2800
-Text GLabel 5350 3200 0    50   Input ~ 0
+Text GLabel 5600 3200 0    50   Input ~ 0
 3_ADC1
 Wire Wire Line
 	3750 2700 3500 2700
-Text GLabel 5350 3100 0    50   Input ~ 0
+Text GLabel 5600 3100 0    50   Input ~ 0
 3_ADC2
 Wire Wire Line
 	3750 2600 3500 2600
-Text GLabel 5350 3000 0    50   Input ~ 0
+Text GLabel 5600 3000 0    50   Input ~ 0
 3_ADC3
 Wire Wire Line
 	3750 2500 3500 2500
-Text GLabel 5350 2900 0    50   Input ~ 0
+Text GLabel 5600 2900 0    50   Input ~ 0
 3_ADC0
 $Comp
@@
 	1    0    0    -1
 $EndComp
-Wire Wire Line
-	5350 3200 5850 3200
-Wire Wire Line
-	5350 3100 5850 3100
-Wire Wire Line
-	5350 3000 5850 3000
-Wire Wire Line
-	5350 2900 5850 2900
 Wire Wire Line
 	3200 6000 2950 6000
@@
 Wire Wire Line
 	1600 1100 1600 1850
-Wire Wire Line
-	1500 1100 1600 1100
 $Comp
 L power:VAA #PWR058
@@
 Text GLabel 1150 4950 0    50   Input ~ 0
 MUXC
-Text GLabel 1000 5050 0    50   Input ~ 0
+Text GLabel 1150 5050 0    50   Input ~ 0
 MUXD
 Text GLabel 1150 5150 0    50   Input ~ 0
@@
 Text GLabel 2950 4900 0    50   Input ~ 0
 MUXC
-Text GLabel 2650 5000 0    50   Input ~ 0
+Text GLabel 2950 5000 0    50   Input ~ 0
 MUXD
 Text GLabel 2950 5100 0    50   Input ~ 0
@@
 	3500 1950 3750 1950
 Wire Wire Line
-	2650 5000 3200 5000
-Wire Wire Line
-	1400 5050 1000 5050
-Connection ~ 1600 1100
-Wire Wire Line
 	2500 2000 2750 2000
 Wire Wire Line
@@
 	6700 6300 6600 6300
 Connection ~ 6600 6300
-Wire Wire Line
-	5050 6300 5000 6300
 Connection ~ 4900 6300
-Connection ~ 5000 6300
 Wire Wire Line
 	5000 6300 4900 6300
@@
 	-1   0    0    1
 $EndComp
-Text GLabel 16050 1650 2    50   Input ~ 0
+Text GLabel 15850 1650 2    50   Input ~ 0
 MUXA1
-Wire Wire Line
-	16050 1650 15600 1650
 Text GLabel 14250 2350 0    50   BiDi ~ 0
 5_OWB_MAIN
@@
 AR Path="/5B9C8983/5BB8E3AD" Ref="U?"  Part="1"
 AR Path="/5BCA1CB6/5BB8E3AD" Ref="U19"  Part="1"
-F 0 "U19" H 15150 3550 60  0000 C CNN
-F 1 "CD74HC4067SM96" H 15150 3444 60  0000 C CNN
+F 0 "U19" H 15800 2350 60  0000 C CNN
+F 1 "CD74HC4067SM96" H 15850 2250 60  0000 C CNN
 F 2 "digikey-footprints:SSOP-24_W5.30mm" H 15400 2450 60  0001 L CNN
 F 3 "http://www.ti.com/lit/ds/symlink/cd74hc4067.pdf" H 15400 2550 60  0001 L CNN
@@
 L power:+5V #PWR?
 U 1 1 5BB8E3B4
-P 15700 1150
+P 15200 1100
 AR Path="/5B9C8983/5BB8E3B4" Ref="#PWR?"  Part="1"
 AR Path="/5BCA1CB6/5BB8E3B4" Ref="#PWR0321"  Part="1"
-F 0 "#PWR0321" H 15700 1000 50  0001 C CNN
-F 1 "+5V" H 15715 1323 50  0000 C CNN
-F 2 "" H 15700 1150 50  0001 C CNN
-F 3 "" H 15700 1150 50  0001 C CNN
-	1    15700 1150
-	1    0    0    -1
-$EndComp
-Wire Wire Line
-	15200 1150 15700 1150
+F 0 "#PWR0321" H 15200 950 50  0001 C CNN
+F 1 "+5V" H 15215 1273 50  0000 C CNN
+F 2 "" H 15200 1100 50  0001 C CNN
+F 3 "" H 15200 1100 50  0001 C CNN
+	1    15200 1100
+	1    0    0    -1
+$EndComp
 Text GLabel 15850 1750 2    50   Input ~ 0
 MUXC
@@
 Wire Wire Line
 	12600 1450 14700 1450
+Text Notes 11100 3500 0    50   ~ 0
+OUTPUT MULTIPLEXING
+Text Notes 12800 2200 0    50   ~ 0
+OWB MULTIPLEXING
+Text Notes 3700 1000 0    50   ~ 0
+IN/ADC MULTIPLEXING
+Wire Wire Line
+	15850 1650 15600 1650
+Wire Wire Line
+	15200 1100 15200 1150
+Wire Wire Line
+	2950 5000 3200 5000
+Wire Wire Line
+	1400 5050 1150 5050
+Wire Wire Line
+	5850 3200 5600 3200
+Wire Wire Line
+	5850 3100 5600 3100
+Wire Wire Line
+	5600 3000 5850 3000
+Wire Wire Line
+	5850 2900 5600 2900
 $EndSCHEMATC

Commit message: USB test instrument support and SCPI support were added to the FW
Parts:
- U1, U16, U2: symbol Analog_Switch:DG408LE -> ANALOGSWITCHES:DG408LE
Changed lines of the file:
@@
 	4050 4750 3950 4750
 $Comp
-L Analog_Switch:DG408LE U2
+L ANALOGSWITCHES:DG408LE U2
 U 1 1 5BA76687
-P 11100 2100
-F 0 "U2" H 11100 2465 50  0000 C CNN
-F 1 "DG408LE" H 11100 2374 50  0000 C CNN
-F 2 "digikey-footprints:SOIC-16_W3.90mm" H 11100 2100 50  0001 C CNN
-F 3 "http://www.vishay.com/docs/78084/dg408le.pdf" H 11100 2100 50  0001 C CNN
-F 4 "DG408LEDY-T1-GE3CT-ND " H 11100 2100 50  0001 C CNN "Digi-Key_PN"
-F 5 "DG408LEDY-T1-GE3" H 0   0   50  0001 C CNN "MPN"
-	1    11100 2100
+P 11100 1800
+F 0 "U2" H 11100 2165 50  0000 C CNN
+F 1 "DG408LE" H 11100 2074 50  0000 C CNN
+F 2 "digikey-footprints:SOIC-16_W3.90mm" H 11100 1800 50  0001 C CNN
+F 3 "http://www.vishay.com/docs/78084/dg408le.pdf" H 11100 1800 50  0001 C CNN
+F 4 "DG408LEDY-T1-GE3CT-ND " H 11100 1800 50  0001 C CNN "Digi-Key_PN"
+F 5 "DG408LEDY-T1-GE3" H 0   -300 50  0001 C CNN "MPN"
+	1    11100 1800
 	1    0    0    -1
 $EndComp
@@
 MUX24
 $Comp
-L Analog_Switch:DG408LE U1
+L ANALOGSWITCHES:DG408LE U1
 U 1 1 5BB6FE9D
-P 9650 4200
-F 0 "U1" H 9650 4550 50  0000 C CNN
-F 1 "DG408LE" H 9650 4450 50  0000 C CNN
-F 2 "digikey-footprints:SOIC-16_W3.90mm" H 9650 4200 50  0001 C CNN
-F 3 "http://www.vishay.com/docs/78084/dg408le.pdf" H 9650 4200 50  0001 C CNN
-F 4 "DG408LEDY-T1-GE3CT-ND " H 0   0   50  0001 C CNN "Digi-Key_PN"
-F 5 "DG408LEDY-T1-GE3" H 0   0   50  0001 C CNN "MPN"
-	1    9650 4200
+P 9650 3900
+F 0 "U1" H 9650 4250 50  0000 C CNN
+F 1 "DG408LE" H 9650 4150 50  0000 C CNN
+F 2 "digikey-footprints:SOIC-16_W3.90mm" H 9650 3900 50  0001 C CNN
+F 3 "http://www.vishay.com/docs/78084/dg408le.pdf" H 9650 3900 50  0001 C CNN
+F 4 "DG408LEDY-T1-GE3CT-ND " H 0   -300 50  0001 C CNN "Digi-Key_PN"
+F 5 "DG408LEDY-T1-GE3" H 0   -300 50  0001 C CNN "MPN"
+	1    9650 3900
 	1    0    0    -1
 $EndComp
@@
 MUX26
 $Comp
-L Analog_Switch:DG408LE U16
+L ANALOGSWITCHES:DG408LE U16
 U 1 1 5BB7C29C
-P 11600 4200
-F 0 "U16" H 11600 4550 50  0000 C CNN
-F 1 "DG408LE" H 11600 4450 50  0000 C CNN
-F 2 "digikey-footprints:SOIC-16_W3.90mm" H 11600 4200 50  0001 C CNN
-F 3 "http://www.vishay.com/docs/78084/dg408le.pdf" H 11600 4200 50  0001 C CNN
-F 4 "DG408LEDY-T1-GE3CT-ND " H 0   0   50  0001 C CNN "Digi-Key_PN"
-F 5 "DG408LEDY-T1-GE3" H 0   0   50  0001 C CNN "MPN"
-	1    11600 4200
+P 11600 3900
+F 0 "U16" H 11600 4250 50  0000 C CNN
+F 1 "DG408LE" H 11600 4150 50  0000 C CNN
+F 2 "digikey-footprints:SOIC-16_W3.90mm" H 11600 3900 50  0001 C CNN
+F 3 "http://www.vishay.com/docs/78084/dg408le.pdf" H 11600 3900 50  0001 C CNN
+F 4 "DG408LEDY-T1-GE3CT-ND " H 0   -300 50  0001 C CNN "Digi-Key_PN"
+F 5 "DG408LEDY-T1-GE3" H 0   -300 50  0001 C CNN "MPN"
+	1    11600 3900
 	1    0    0    -1
 $EndComp
