File: QualificationTestingAutomation/SchematicAutomation/ATMEGA2560.sch (KiCad schematic (older format))
At the start: 18 parts, among them J12 0015912120, U3 AT90USB1287-AU, Y1 16MHz

Commit message: C WPCB was started and the schematic is full, I am thinking of implementing the UART test using analog muxes.
Parts:
- C1, C2, C3, C4, C5: footprint digikey-footprints:0603 -> smt:C-0603
- R171, R172, R173, R175, R3, R4: footprint digikey-footprints:0603 -> Resistor_SMD:R_0402_1005Metric
- R174: value 10K -> 50K; footprint digikey-footprints:0603 -> Resistor_SMD:R_0402_1005Metric
- R176: value 10K -> 100K; footprint digikey-footprints:0603 -> Resistor_SMD:R_0402_1005Metric
- Y1: Category (none) -> Clocks; Digi-Key_PN (none) -> 535-10226-1-ND
Connections:
- wire segments 105 -> 104
Other:
- moved on the sheet: U3

Commit message: the PCB is complete and has been ordered
Parts:
- L1: footprint digikey-footprints:0603 -> digikey-footprints:0805
Connections:
- net labels added: CTS_CONT, TX_CONT
- wire segments 104 -> 107
Changed lines of the file:
@@
 F 0 "L1" V 5250 2350 60  0000 L CNB
 F 1 "10uH" V 5350 2300 40  0000 L CNN
-F 2 "digikey-footprints:0603" H 5500 2220 40  0001 C CNN
+F 2 "digikey-footprints:0805" H 5500 2220 40  0001 C CNN
 F 3 "https://search.murata.co.jp/Ceramy/image/img/P02/JELF243B-0012.pdf" V 6750 4600 60  0000 C CNN
 F 4 "490-4025-1-ND" H 5500 2515 45  0001 C CNN "PART"
@@
 L dk_Rectangular-Connectors-Headers-Male-Pins:0015912120 J12
 U 1 1 5B913E87
-P 3450 6000
-F 0 "J12" H 3450 6447 60  0000 C CNN
-F 1 "0015912120" H 3450 6341 60  0000 C CNN
-F 2 "digikey-footprints:PinHeader_2x6_P2.54mm_Vertical_SMD" H 3650 6200 60  0001 L CNN
-F 3 "https://www.molex.com/pdm_docs/sd/015912120_sd.pdf" H 3650 6300 60  0001 L CNN
-F 4 "WM17452-ND" H 3650 6400 60  0001 L CNN "Digi-Key_PN"
-F 5 "0015912120" H 3650 6500 60  0001 L CNN "MPN"
-F 6 "Connectors, Interconnects" H 3650 6600 60  0001 L CNN "Category"
-F 7 "Rectangular Connectors - Headers, Male Pins" H 3650 6700 60  0001 L CNN "Family"
-F 8 "https://www.molex.com/pdm_docs/sd/015912120_sd.pdf" H 3650 6800 60  0001 L CNN "DK_Datasheet_Link"
-F 9 "/product-detail/en/molex-connector-corporation/0015912120/WM17452-ND/614768" H 3650 6900 60  0001 L CNN "DK_Detail_Page"
-F 10 "CONN HEADER 12POS .100 VERT TIN" H 3650 7000 60  0001 L CNN "Description"
-F 11 "Molex Connector Corporation" H 3650 7100 60  0001 L CNN "Manufacturer"
-F 12 "Active" H 3650 7200 60  0001 L CNN "Status"
-	1    3450 6000
-	1    0    0    -1
+P 3350 6600
+F 0 "J12" H 3350 7047 60  0000 C CNN
+F 1 "0015912120" H 3350 6941 60  0000 C CNN
+F 2 "digikey-footprints:PinHeader_2x6_P2.54mm_Vertical_SMD" H 3550 6800 60  0001 L CNN
+F 3 "https://www.molex.com/pdm_docs/sd/015912120_sd.pdf" H 3550 6900 60  0001 L CNN
+F 4 "WM17452-ND" H 3550 7000 60  0001 L CNN "Digi-Key_PN"
+F 5 "0015912120" H 3550 7100 60  0001 L CNN "MPN"
+F 6 "Connectors, Interconnects" H 3550 7200 60  0001 L CNN "Category"
+F 7 "Rectangular Connectors - Headers, Male Pins" H 3550 7300 60  0001 L CNN "Family"
+F 8 "https://www.molex.com/pdm_docs/sd/015912120_sd.pdf" H 3550 7400 60  0001 L CNN "DK_Datasheet_Link"
+F 9 "/product-detail/en/molex-connector-corporation/0015912120/WM17452-ND/614768" H 3550 7500 60  0001 L CNN "DK_Detail_Page"
+F 10 "CONN HEADER 12POS .100 VERT TIN" H 3550 7600 60  0001 L CNN "Description"
+F 11 "Molex Connector Corporation" H 3550 7700 60  0001 L CNN "Manufacturer"
+F 12 "Active" H 3550 7800 60  0001 L CNN "Status"
+	1    3350 6600
+	0    -1   -1   0
 $EndComp
 Wire Wire Line
 	4800 6250 4800 6300
 Wire Wire Line
-	4800 6300 3650 6300
-Wire Wire Line
 	4800 6150 4800 6200
 Wire Wire Line
-	4800 6200 3650 6200
-Wire Wire Line
 	4800 6050 4800 6100
 Wire Wire Line
-	4800 6100 3650 6100
-Wire Wire Line
 	4800 5950 4800 6000
-Wire Wire Line
-	4800 6000 3650 6000
 Wire Wire Line
 	4800 5850 4800 5900
@@
 TCK
 Wire Wire Line
-	3650 5900 3750 5900
+	3650 6400 3750 6400
 $Comp
 L power:GND #PWR016
 U 1 1 5B9183F6
-P 3850 5900
-F 0 "#PWR016" H 3850 5650 50  0001 C CNN
-F 1 "GND" H 3855 5727 50  0000 C CNN
-F 2 "" H 3850 5900 50  0001 C CNN
-F 3 "" H 3850 5900 50  0001 C CNN
-	1    3850 5900
-	1    0    0    -1
-$EndComp
-Wire Wire Line
-	3650 5800 4000 5800
+P 3850 6400
+F 0 "#PWR016" H 3850 6150 50  0001 C CNN
+F 1 "GND" H 3855 6227 50  0000 C CNN
+F 2 "" H 3850 6400 50  0001 C CNN
+F 3 "" H 3850 6400 50  0001 C CNN
+	1    3850 6400
+	1    0    0    -1
+$EndComp
+Wire Wire Line
+	3650 6800 4000 6800
 $Comp
 L power:+3V3 #PWR018
 U 1 1 5B919423
-P 4000 5800
-F 0 "#PWR018" H 4000 5650 50  0001 C CNN
-F 1 "+3V3" H 4015 5973 50  0000 C CNN
-F 2 "" H 4000 5800 50  0001 C CNN
-F 3 "" H 4000 5800 50  0001 C CNN
-	1    4000 5800
+P 4000 6800
+F 0 "#PWR018" H 4000 6650 50  0001 C CNN
+F 1 "+3V3" H 4015 6973 50  0000 C CNN
+F 2 "" H 4000 6800 50  0001 C CNN
+F 3 "" H 4000 6800 50  0001 C CNN
+	1    4000 6800
 	-1   0    0    1
 $EndComp
 Wire Wire Line
-	3250 5900 3150 5900
-Wire Wire Line
-	3250 6000 3150 6000
-Text HLabel 3150 6000 0    50   Input ~ 0
+	3450 6800 3450 6900
+Text HLabel 3450 6350 1    50   Input ~ 0
 D-
-Text HLabel 3150 5900 0    50   Input ~ 0
+Text HLabel 3450 6900 3    50   Input ~ 0
 D+
-Wire Wire Line
-	3250 6100 3150 6100
-Text HLabel 3150 6100 0    50   Input ~ 0
+Text HLabel 3550 6800 3    50   Input ~ 0
 VBUS
 Wire Wire Line
-	3250 5800 3250 5850
-Wire Wire Line
-	3250 5850 3750 5850
-Wire Wire Line
-	3750 5850 3750 5900
-Connection ~ 3750 5900
-Wire Wire Line
-	3750 5900 3850 5900
+	3750 6350 3750 6400
+Connection ~ 3750 6400
+Wire Wire Line
+	3750 6400 3850 6400
 Text GLabel 6250 4650 2    50   Input ~ 0
 MUX26
@@
 NoConn ~ 6000 4450
 NoConn ~ 6000 4950
-NoConn ~ 6000 5050
-NoConn ~ 6000 5150
 NoConn ~ 6000 5250
 NoConn ~ 6000 5350
@@
 Wire Wire Line
 	5600 2500 5650 2500
-NoConn ~ 3250 6200
-NoConn ~ 3250 6300
 Text GLabel 6350 5950 2    50   Input ~ 0
 MUXA1
@@
 Wire Wire Line
 	6350 6050 6000 6050
+Text GLabel 6000 5050 2    50   Input ~ 0
+TX_CONT
+Text GLabel 6000 5150 2    50   Input ~ 0
+CTS_CONT
+Wire Wire Line
+	3350 6300 3350 6400
+Wire Wire Line
+	3350 6300 4800 6300
+Wire Wire Line
+	3300 6200 3300 6800
+Wire Wire Line
+	3300 6800 3350 6800
+Wire Wire Line
+	3300 6200 4800 6200
+Wire Wire Line
+	3250 6100 3250 6400
+Wire Wire Line
+	3250 6100 4800 6100
+Wire Wire Line
+	3450 6350 3450 6400
+NoConn ~ 3200 6400
+NoConn ~ 3150 6400
+NoConn ~ 3150 6800
+NoConn ~ 3550 6400
+Wire Wire Line
+	2750 6800 2750 6000
+Wire Wire Line
+	2750 6000 4800 6000
+Wire Wire Line
+	2750 6800 3250 6800
 $EndSCHEMATC

Commit message: Added Schematic Libraries
Parts:
- added S4: 1825910-6, digikey-footprints:Switch_Tactile_THT_6x6mm, symbol dk_Tactile-Switches:1825910-6
Connections:
- wire segments 107 -> 116
Changed lines of the file:
@@
 	3800 4850 4800 4850
 Wire Wire Line
-	2100 5500 3800 5500
+	2100 5500 2250 5500
 $Comp
 L power:+12V #PWR0312
@@
 Wire Wire Line
 	2750 6800 3250 6800
+$Comp
+L dk_Tactile-Switches:1825910-6 S4
+U 1 1 5BA88744
+P 1450 4850
+F 0 "S4" H 1450 5197 60  0000 C CNN
+F 1 "1825910-6" H 1450 5091 60  0000 C CNN
+F 2 "digikey-footprints:Switch_Tactile_THT_6x6mm" H 1650 5050 60  0001 L CNN
+F 3 "http://www.te.com/commerce/DocumentDelivery/DDEController?Action=srchrtrv&DocNm=1825910&DocType=Customer+Drawing&DocLang=English" H 1650 5150 60  0001 L CNN
+F 4 "450-1650-ND" H 1650 5250 60  0001 L CNN "Digi-Key_PN"
+F 5 "1825910-6" H 1650 5350 60  0001 L CNN "MPN"
+F 6 "Switches" H 1650 5450 60  0001 L CNN "Category"
+F 7 "Tactile Switches" H 1650 5550 60  0001 L CNN "Family"
+F 8 "http://www.te.com/commerce/DocumentDelivery/DDEController?Action=srchrtrv&DocNm=1825910&DocType=Customer+Drawing&DocLang=English" H 1650 5650 60  0001 L CNN "DK_Datasheet_Link"
+F 9 "/product-detail/en/te-connectivity-alcoswitch-switches/1825910-6/450-1650-ND/1632536" H 1650 5750 60  0001 L CNN "DK_Detail_Page"
+F 10 "SWITCH TACTILE SPST-NO 0.05A 24V" H 1650 5850 60  0001 L CNN "Description"
+F 11 "TE Connectivity ALCOSWITCH Switches" H 1650 5950 60  0001 L CNN "Manufacturer"
+F 12 "Active" H 1650 6050 60  0001 L CNN "Status"
+	1    1450 4850
+	1    0    0    -1
+$EndComp
+Wire Wire Line
+	2250 5500 2250 5150
+Wire Wire Line
+	2250 5150 1650 5150
+Wire Wire Line
+	1650 5150 1650 4950
+Connection ~ 2250 5500
+Wire Wire Line
+	2250 5500 3800 5500
+Connection ~ 1650 4950
+Wire Wire Line
+	1650 4950 1650 4750
+Wire Wire Line
+	1250 4950 1250 4900
+Wire Wire Line
+	1250 4900 1000 4900
+Wire Wire Line
+	1000 4900 1000 5100
+Connection ~ 1250 4900
+Wire Wire Line
+	1250 4900 1250 4750
+$Comp
+L power:GND #PWR0283
+U 1 1 5BA9B235
+P 1000 5100
+F 0 "#PWR0283" H 1000 4850 50  0001 C CNN
+F 1 "GND" H 1005 4927 50  0000 C CNN
+F 2 "" H 1000 5100 50  0001 C CNN
+F 3 "" H 1000 5100 50  0001 C CNN
+	1    1000 5100
+	1    0    0    -1
+$EndComp
 $EndSCHEMATC

Commit message: CLEANED UP THE SCHEMATICS ADDED NEADED FIXES FOUND ON THE BOARD
Connections:
- wire segments 116 -> 115
- no-connect marks 23 -> 22
Other:
- note added: "ADC/IN MUX SELECT"
- note added: "ADC/IN/OUT port MUXING SELECT"
- note added: "BOOTLOADER enable button"
- note added: "OUT Muxing select"
- note added: "PWR ON RELAY SELECT"
- note added: "RESET BUTTON"
- note added: "SHOULD PROBABLY MAKE IT AS A STANDARD JTAG CONNECTOR"
- note added: "UART PORTS"

Commit message: USB test instrument support and SCPI support were added to the FW
Connections:
- wire segments 115 -> 113
Changed lines of the file:
@@
 Text Label 4250 6000 0    50   ~ 0
 TCK
-Wire Wire Line
-	3650 6400 3750 6400
 $Comp
 L power:GND #PWR016
@@
 Text HLabel 3550 6800 3    50   Input ~ 0
 VBUS
-Wire Wire Line
-	3750 6350 3750 6400
-Connection ~ 3750 6400
-Wire Wire Line
-	3750 6400 3850 6400
 Text GLabel 6250 4650 2    50   Input ~ 0
 MUX26
@@
 	3850 5150 3850 5250
 $Comp
-L power:GND #PWR?
+L power:GND #PWR0283
 U 1 1 5BCB7C6E
 P 3600 5150
-F 0 "#PWR?" H 3600 4900 50  0001 C CNN
+F 0 "#PWR0283" H 3600 4900 50  0001 C CNN
 F 1 "GND" H 3605 4977 50  0000 C CNN
 F 2 "" H 3600 5150 50  0001 C CNN
@@
 	1    0    0    -1
 $EndComp
+Wire Wire Line
+	3650 6400 3850 6400
 $EndSCHEMATC

Commit message: RX TX mixup was solved by changing RX_3V3 and TX_3V3 on the XOR side Same goes for CTS and RTS and some general clean up
Signed-off-by: Riyad Alalami <riyadhelalami@gmail.com>
Connections:
- wire segments 113 -> 114
Changed lines of the file:
@@
 	3350 6300 3350 6400
 Wire Wire Line
-	3350 6300 4800 6300
-Wire Wire Line
-	3300 6200 3300 6800
-Wire Wire Line
-	3300 6800 3350 6800
-Wire Wire Line
-	3300 6200 4800 6200
-Wire Wire Line
 	3250 6100 3250 6400
 Wire Wire Line
@@
 Wire Wire Line
 	3650 6400 3850 6400
+Wire Wire Line
+	3350 7150 3350 6800
+Wire Wire Line
+	3350 6300 4800 6300
+Wire Wire Line
+	4800 5900 4650 5900
+Wire Wire Line
+	4650 5900 4650 7150
+Wire Wire Line
+	4650 7150 3350 7150
 $EndSCHEMATC
