File: QualificationTestingAutomation/The Matrix Modular/Switchero Module/SwitcheroModule/RX.sch (KiCad schematic (older format))
At the start: 2 parts, among them U12 CD4070B

Commit message: Cleaned up the libraries Cleaned up the tracks Adjusted footprints to the manufacturers minimum size.
Parts:
- C2: symbol TheMatrix-rescue:CAP-passive-SchematicAutomation-rescue -> SwitcheroModule-rescue:CAP-passive-SchematicAutomation-rescue-TheMatrix-rescue
- U12: symbol TheMatrix-rescue:CD4070B-4XXXSeriesLOGIC-SchematicAutomation-rescue -> SwitcheroModule-rescue:CD4070B-4XXXSeriesLOGIC-SchematicAutomation-rescue-TheMatrix-rescue
Changed lines of the file:
@@
 $EndBitmap
 $Comp
-L TheMatrix-rescue:CD4070B-4XXXSeriesLOGIC-SchematicAutomation-rescue U?
+L SwitcheroModule-rescue:CD4070B-4XXXSeriesLOGIC-SchematicAutomation-rescue-TheMatrix-rescue U?
 U 1 1 5CA21608
 P 6050 1050
@@
 	2800 1400 2650 1400
 $Comp
-L TheMatrix-rescue:CAP-passive-SchematicAutomation-rescue C?
+L SwitcheroModule-rescue:CAP-passive-SchematicAutomation-rescue-TheMatrix-rescue C?
 U 1 1 5CAEB1E7
 P 7050 1300
