File: QualificationTestingAutomation/The Matrix Modular/Switchero Module/SwitcheroModule/UART.sch (KiCad schematic (older format))
At the start: 26 parts, among them Q10 2N7002DW, Q2 2N7002DW, Q5 2N7002DW, Q8 2N7002DW, U11 MAX324CUA, U12 CD4070B, U15 MAX324CUA

Commit message: Cleaned up the libraries Cleaned up the tracks Adjusted footprints to the manufacturers minimum size.
Parts:
- C7: symbol TheMatrix-rescue:CAP-passive-SchematicAutomation-rescue -> SwitcheroModule-rescue:CAP-passive-SchematicAutomation-rescue-TheMatrix-rescue
- Q10, Q2, Q5, Q8: symbol TheMatrix-rescue:2N7002DW-dk_Transistors-FETs-MOSFETs-Arrays-SchematicAutomation-rescue -> SwitcheroModule-rescue:2N7002DW-dk_Transistors-FETs-MOSFETs-Arrays-SchematicAutomation-rescue-TheMatrix-rescue
- R10, R12, R21, R29, R30, R31, R32, R33, R34, R38, R40, R42, R47, R49, R51, R53, R8: symbol TheMatrix-rescue:RESISTOR-passive-SchematicAutomation-rescue -> SwitcheroModule-rescue:RESISTOR-passive-SchematicAutomation-rescue-TheMatrix-rescue
- U12: symbol TheMatrix-rescue:CD4070B-4XXXSeriesLOGIC-SchematicAutomation-rescue -> SwitcheroModule-rescue:CD4070B-4XXXSeriesLOGIC-SchematicAutomation-rescue-TheMatrix-rescue
Changed lines of the file:
@@
 $EndDescr
 $Comp
-L TheMatrix-rescue:2N7002DW-dk_Transistors-FETs-MOSFETs-Arrays-SchematicAutomation-rescue Q?
+L SwitcheroModule-rescue:2N7002DW-dk_Transistors-FETs-MOSFETs-Arrays-SchematicAutomation-rescue-TheMatrix-rescue Q?
 U 1 1 5C46C762
 P 3450 4500
@@
 AR Path="/5C90F514/5C94BFB1/5C46C762" Ref="Q2"  Part="1"
 AR Path="/5C90F514/5C94ECF2/5C46C762" Ref="Q6"  Part="1"
+AR Path="/5C46C762" Ref="Q6"  Part="1"
 F 0 "Q6" H 3450 4987 60  0000 C CNN
 F 1 "2N7002DW" H 3450 4881 60  0000 C CNN
@@
 $EndComp
 $Comp
-L TheMatrix-rescue:RESISTOR-passive-SchematicAutomation-rescue R?
+L SwitcheroModule-rescue:RESISTOR-passive-SchematicAutomation-rescue-TheMatrix-rescue R?
 U 1 1 5C46C76E
 P 4200 4300
@@
 Connection ~ 2850 4900
 $Comp
-L TheMatrix-rescue:RESISTOR-passive-SchematicAutomation-rescue R?
+L SwitcheroModule-rescue:RESISTOR-passive-SchematicAutomation-rescue-TheMatrix-rescue R?
 U 1 1 5C46C789
 P 2400 4900
@@
 	2150 4300 3150 4300
 $Comp
-L TheMatrix-rescue:2N7002DW-dk_Transistors-FETs-MOSFETs-Arrays-SchematicAutomation-rescue Q?
+L SwitcheroModule-rescue:2N7002DW-dk_Transistors-FETs-MOSFETs-Arrays-SchematicAutomation-rescue-TheMatrix-rescue Q?
 U 1 1 5BC141FA
 P 9350 4400
@@
 AR Path="/5C90F514/5C94BFB1/5BC141FA" Ref="Q5"  Part="1"
 AR Path="/5C90F514/5C94ECF2/5BC141FA" Ref="Q9"  Part="1"
+AR Path="/5BC141FA" Ref="Q9"  Part="1"
 F 0 "Q9" H 9350 4887 60  0000 C CNN
 F 1 "2N7002DW" H 9350 4781 60  0000 C CNN
@@
 	9050 4200 8850 4200
 $Comp
-L TheMatrix-rescue:RESISTOR-passive-SchematicAutomation-rescue R?
+L SwitcheroModule-rescue:RESISTOR-passive-SchematicAutomation-rescue-TheMatrix-rescue R?
 U 1 1 5BC14205
 P 8600 4200
@@
 Connection ~ 9950 4800
 $Comp
-L TheMatrix-rescue:RESISTOR-passive-SchematicAutomation-rescue R?
+L SwitcheroModule-rescue:RESISTOR-passive-SchematicAutomation-rescue-TheMatrix-rescue R?
 U 1 1 5BC14215
 P 10400 4800
@@
 	5400 4600 5350 4600
 $Comp
-L TheMatrix-rescue:RESISTOR-passive-SchematicAutomation-rescue R?
+L SwitcheroModule-rescue:RESISTOR-passive-SchematicAutomation-rescue-TheMatrix-rescue R?
 U 1 1 5BBE173B
 P 4450 4450
@@
 	7700 4500 7950 4500
 $Comp
-L TheMatrix-rescue:RESISTOR-passive-SchematicAutomation-rescue R?
+L SwitcheroModule-rescue:RESISTOR-passive-SchematicAutomation-rescue-TheMatrix-rescue R?
 U 1 1 5BBEA4F3
 P 8450 5150
@@
 BIAS RESISTORS
 $Comp
-L TheMatrix-rescue:RESISTOR-passive-SchematicAutomation-rescue R?
+L SwitcheroModule-rescue:RESISTOR-passive-SchematicAutomation-rescue-TheMatrix-rescue R?
 U 1 1 5BC0A9BF
 P 4250 4750
@@
 WE SHOULD ADD MORE DECOUPLING CAPS
 $Comp
-L TheMatrix-rescue:CD4070B-4XXXSeriesLOGIC-SchematicAutomation-rescue U?
+L SwitcheroModule-rescue:CD4070B-4XXXSeriesLOGIC-SchematicAutomation-rescue-TheMatrix-rescue U?
 U 1 1 5C46C7B8
 P 6200 2400
@@
 $EndComp
 $Comp
-L TheMatrix-rescue:RESISTOR-passive-SchematicAutomation-rescue R?
+L SwitcheroModule-rescue:RESISTOR-passive-SchematicAutomation-rescue-TheMatrix-rescue R?
 U 1 1 5CACEC46
 P 4450 4600
@@
 Connection ~ 4100 4600
 $Comp
-L TheMatrix-rescue:RESISTOR-passive-SchematicAutomation-rescue R?
+L SwitcheroModule-rescue:RESISTOR-passive-SchematicAutomation-rescue-TheMatrix-rescue R?
 U 1 1 5CAD91E6
 P 8650 4500
@@
 Connection ~ 8800 4500
 $Comp
-L TheMatrix-rescue:2N7002DW-dk_Transistors-FETs-MOSFETs-Arrays-SchematicAutomation-rescue Q?
+L SwitcheroModule-rescue:2N7002DW-dk_Transistors-FETs-MOSFETs-Arrays-SchematicAutomation-rescue-TheMatrix-rescue Q?
 U 1 1 5CA361A5
 P 2750 3150
@@
 AR Path="/5C90F514/5C94BFB1/5CA361A5" Ref="Q?"  Part="1"
 AR Path="/5C90F514/5C94ECF2/5CA361A5" Ref="Q8"  Part="1"
+AR Path="/5CA361A5" Ref="Q8"  Part="1"
 F 0 "Q8" H 2750 3637 60  0000 C CNN
 F 1 "2N7002DW" H 2750 3531 60  0000 C CNN
@@
 $EndComp
 $Comp
-L TheMatrix-rescue:RESISTOR-passive-SchematicAutomation-rescue R?
+L SwitcheroModule-rescue:RESISTOR-passive-SchematicAutomation-rescue-TheMatrix-rescue R?
 U 1 1 5CA361AE
 P 3500 2950
@@
 Connection ~ 2150 3550
 $Comp
-L TheMatrix-rescue:RESISTOR-passive-SchematicAutomation-rescue R?
+L SwitcheroModule-rescue:RESISTOR-passive-SchematicAutomation-rescue-TheMatrix-rescue R?
 U 1 1 5CA361BE
 P 1700 3550
@@
 	4700 3250 4650 3250
 $Comp
-L TheMatrix-rescue:RESISTOR-passive-SchematicAutomation-rescue R?
+L SwitcheroModule-rescue:RESISTOR-passive-SchematicAutomation-rescue-TheMatrix-rescue R?
 U 1 1 5CA361F6
 P 3750 3100
@@
 	3400 3100 3400 3250
 $Comp
-L TheMatrix-rescue:RESISTOR-passive-SchematicAutomation-rescue R?
+L SwitcheroModule-rescue:RESISTOR-passive-SchematicAutomation-rescue-TheMatrix-rescue R?
 U 1 1 5CA36201
 P 3550 3400
@@
 SHOULD WE ADD BIASING RESISTORS JUST IN CASE
 $Comp
-L TheMatrix-rescue:RESISTOR-passive-SchematicAutomation-rescue R?
+L SwitcheroModule-rescue:RESISTOR-passive-SchematicAutomation-rescue-TheMatrix-rescue R?
 U 1 1 5CA36212
 P 3750 3250
@@
 RS232INV
 $Comp
-L TheMatrix-rescue:2N7002DW-dk_Transistors-FETs-MOSFETs-Arrays-SchematicAutomation-rescue Q?
+L SwitcheroModule-rescue:2N7002DW-dk_Transistors-FETs-MOSFETs-Arrays-SchematicAutomation-rescue-TheMatrix-rescue Q?
 U 1 1 5CA446D5
 P 10650 3050
@@
 AR Path="/5C90F514/5C94BFB1/5CA446D5" Ref="Q?"  Part="1"
 AR Path="/5C90F514/5C94ECF2/5CA446D5" Ref="Q10"  Part="1"
+AR Path="/5CA446D5" Ref="Q10"  Part="1"
 F 0 "Q10" H 10650 3537 60  0000 C CNN
 F 1 "2N7002DW" H 10650 3431 60  0000 C CNN
@@
 	10350 2850 10150 2850
 $Comp
-L TheMatrix-rescue:RESISTOR-passive-SchematicAutomation-rescue R?
+L SwitcheroModule-rescue:RESISTOR-passive-SchematicAutomation-rescue-TheMatrix-rescue R?
 U 1 1 5CA446DF
 P 9900 2850
@@
 Connection ~ 11250 3450
 $Comp
-L TheMatrix-rescue:RESISTOR-passive-SchematicAutomation-rescue R?
+L SwitcheroModule-rescue:RESISTOR-passive-SchematicAutomation-rescue-TheMatrix-rescue R?
 U 1 1 5CA446EE
 P 11700 3450
@@
 	9000 3150 9250 3150
 $Comp
-L TheMatrix-rescue:RESISTOR-passive-SchematicAutomation-rescue R?
+L SwitcheroModule-rescue:RESISTOR-passive-SchematicAutomation-rescue-TheMatrix-rescue R?
 U 1 1 5CA44728
 P 9750 3800
@@
 THESE SHORTS are to bypass the switch
 $Comp
-L TheMatrix-rescue:RESISTOR-passive-SchematicAutomation-rescue R?
+L SwitcheroModule-rescue:RESISTOR-passive-SchematicAutomation-rescue-TheMatrix-rescue R?
 U 1 1 5CA44735
 P 9950 3150
@@
 	8450 2400 10150 2400
 $Comp
-L TheMatrix-rescue:CAP-passive-SchematicAutomation-rescue C?
+L SwitcheroModule-rescue:CAP-passive-SchematicAutomation-rescue-TheMatrix-rescue C?
 U 1 1 5CAEB908
 P 7200 2700
