File: QualificationTestingAutomation/The Matrix Modular/Switchero Module/SwitcheroModule/_saved_Micro.sch (KiCad schematic (older format))
At the start: 10 parts, among them SW1 SW_DIP_x04, U1 TC2050-JTAG-SchematicAutomati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, U2 AT25SF081-SSHD-X, U3 MSP430G2755IRHA40, U4 SN74HC266DR, U5 SN74LVC08APWR

Commit message: Updated the layout to accomodate the voltage and current sensing.
Connections:
- net A5: now also U3.26 (P3.7/A6/TA1.2); no longer U3.40 (TA1.0/ROSC/P2.5)
- net \HOLD: now also U3.40 (TA1.0/ROSC/P2.5); no longer U3.26 (P3.7/A6/TA1.2)
Changed lines of the file:
@@
 Text GLabel 6250 4550 2    50   Input ~ 0
 A2
-Text Label 3700 5050 2    50   ~ 0
+Text Label 6250 4850 0    50   ~ 0
 \HOLD
 Wire Wire Line
@@
 Wire Wire Line
 	5050 5300 4800 5300
-Text GLabel 6250 4850 2    50   Input ~ 0
+Text GLabel 3700 5050 0    50   Input ~ 0
 A5
 $Comp
-L power:+2V5 #PWR?
+L power:+2V5 #PWR0182
 U 1 1 5CA7FFF6
 P 6250 4750
-F 0 "#PWR?" H 6250 4600 50  0001 C CNN
+F 0 "#PWR0182" H 6250 4600 50  0001 C CNN
 F 1 "+2V5" V 6265 4878 50  0000 L CNN
 F 2 "" H 6250 4750 50  0001 C CNN
@@
 $EndComp
 $Comp
-L power:GND #PWR?
+L power:GND #PWR0216
 U 1 1 5CA8286A
 P 6250 4650
-F 0 "#PWR?" H 6250 4400 50  0001 C CNN
+F 0 "#PWR0216" H 6250 4400 50  0001 C CNN
 F 1 "GND" H 6255 4477 50  0000 C CNN
 F 2 "" H 6250 4650 50  0001 C CNN
