File: QualificationTestingAutomation/The Matrix Modular/ModularMatrix/PWR.sch (KiCad schematic (older format))
At the start: 61 parts, among them J3 Barrel_Jack_MountingPin, U1 TPS563210, U2 LT8361, U3 TPS563210, U4 TLV70018_SOT23-5, U5 LM2776, U6 LM2776

Commit message: Schematic Clean ups the layout needs to be changed
Parts:
- R11, R12: value 25.5K -> 0
Other:
- note added: "Change to a viahole"
- moved on the sheet: C22, C26, C31, C32, C34, C35, C44, C45, C46, C49, U4
